File: GMK67-HE_Trial.kicad_pcb (KiCad board)
At the start: 2 copper layers, 301.9 x 162.3 mm, 208 parts, among them U1 Hall_Sensor, U10 Hall_Sensor, U11 Hall_Sensor, U12 Hall_Sensor, U13 Hall_Sensor, U14 Hall_Sensor, U15 Hall_Sensor, U16 Hall_Sensor, U17 Hall_Sensor, U18 Hall_Sensor, U19 Hall_Sensor, U2 Hall_Sensor, U20 Hall_Sensor, U21 Hall_Sensor, U22 Hall_Sensor, U23 Hall_Sensor, U24 Hall_Sensor, U25 Hall_Sensor, U26 Hall_Sensor, U27 Hall_Sensor, U28 Hall_Sensor, U29 Hall_Sensor, U3 Hall_Sensor, U30 Hall_Sensor, U31 Hall_Sensor, U32 Hall_Sensor, U33 Hall_Sensor, U34 Hall_Sensor, U35 Hall_Sensor, U36 Hall_Sensor, U37 Hall_Sensor, U38 Hall_Sensor, U39 Hall_Sensor, U4 Hall_Sensor, U40 Hall_Sensor, U41 Hall_Sensor, U42 Hall_Sensor, U43 Hall_Sensor, U44 Hall_Sensor, U45 Hall_Sensor, U46 Hall_Sensor, U47 Hall_Sensor, U48 Hall_Sensor, U49 Hall_Sensor, U5 Hall_Sensor, U50 Hall_Sensor, U51 Hall_Sensor, U52 Hall_Sensor, U53 Hall_Sensor, U54 Hall_Sensor, U55 Hall_Sensor, U56 Hall_Sensor, U57 Hall_Sensor, U58 Hall_Sensor, U59 Hall_Sensor, U6 Hall_Sensor, U60 Hall_Sensor, U61 Hall_Sensor, U62 Hall_Sensor, U63 Hall_Sensor, U64 Hall_Sensor, U65 Hall_Sensor, U66 Hall_Sensor, U7 Hall_Sensor, U8 Hall_Sensor, U9 Hall_Sensor

Commit message: Second Commit
new wiring and label
Parts:
- removed AM4:10: Enter, HE_Keyswitch:MX_Gateron_HE_2.25u_Stab
- removed C20, C21: 10µF, ScottoKeebs_Components:Capacitor_0402
- removed C22: 1µF, ScottoKeebs_Components:Capacitor_0402
- removed C23: 100nF, ScottoKeebs_Components:Capacitor_0402
- removed ICC1: TP4057, Package_TO_SOT_SMD:SOT-23-6
- removed L1: 1uF, Inductor_SMD:L_0402_1005Metric
- removed LED3: CLV1L-FKB, LED_SMD:LED_Cree-PLCC4_3.2x2.8mm_CCW
- removed PR1: LM3670MF, Package_TO_SOT_SMD:TSOT-23-5
- removed R12: 1.6k, ScottoKeebs_Components:Resistor_0402
- removed SD1: BAT54C, Package_TO_SOT_SMD:SOT-23
- added AM4:13: Left, HE_Keyswitch:MX_Gateron_HE_1u, F.Cu at (304.7, 151.7)
- AM4:11: value R Shift -> Enter; footprint HE_Keyswitch:MX_Gateron_HE_1.75u -> HE_Keyswitch:MX_Gateron_HE_2.25u_Stab
- AM4:12: value Left -> R Shift; footprint HE_Keyswitch:MX_Gateron_HE_1u -> HE_Keyswitch:MX_Gateron_HE_1.75u
- C1: value 4.7uF -> 1µF
- C2: value 10uF -> 100nF
- R11: value 1k -> 250k
- moved R11 72.0 mm to (142.8, 230.8), turned to 90 degrees
- moved C2 58.5 mm to (130.9, 226.1), turned to 180 degrees
- moved AM4:12 52.8 mm to (297.5, 132.7)
- moved C1 50.5 mm to (130.9, 224.9), turned to 180 degrees
- moved AM4:11 41.4 mm to (311.8, 113.6)
- moved LED1 38.3 mm to (290.4, 148.5)
- moved AM1:1 34.7 mm to (178.4, 151.7)
- moved AM1:11 34.7 mm to (128.4, 113.6)
- moved AM1:2 34.7 mm to (166.5, 113.6)
- moved AM2:13 34.7 mm to (185.6, 113.6)
- moved AM2:2 34.7 mm to (223.7, 113.6)
- moved AM3 34.7 mm to (266.4, 104.1)
- moved AM3:1 34.7 mm to (273.7, 151.7)
- moved AM3:14 34.7 mm to (249.9, 151.7)
- moved AM3:15 34.7 mm to (261.8, 113.6)
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Connections:
- AM4 pad 18: GND -> AM4:13
- AM4 pad 21: AM4:10 -> GND
- C1 pad 2: Net-(PR1-EN) -> Net-(ESD1-VCC)
- C12 pad 2: VDD A22 -> 3.3V
- C13 pad 2: VDD A22 -> 3.3V
- C14 pad 2: VDD A22 -> 3.3V
- C15 pad 2: VDD A22 -> 3.3V
- C16 pad 2: VDD A22 -> 3.3V
- C2 pad 2: 3.3V -> Net-(ESD1-VCC)
- DBG3 pad 1: VDD A22 -> 3.3V
- ICCPR1 pad 16: unconnected-(ICCPR1-VSET2-Pad16) -> Net-(ICCPR1-VSET2)
- ICCPR1 pad 17: unconnected-(ICCPR1-VSET1-Pad17) -> GND
- ICCPR1 pad 20: unconnected-(ICCPR1-VSYS-Pad20) -> VSYS
- ICCPR1 pad 25: unconnected-(ICCPR1-LED0-Pad25) -> LED0
- ICCPR1 pad 26: unconnected-(ICCPR1-LED1-Pad26) -> LED1
- ICCPR1 pad 27: unconnected-(ICCPR1-LED2-Pad27) -> LED2
- ICCPR1 pad 32: VDD A22 -> 3.3V
- LED1 pad 1: Net-(LED1-A) -> GND
- LED1 pad 2: Net-(ICC1-~{CHRG}) -> MCU R
- LED1 pad 3: Net-(ICC1-STDBY) -> MCU G
- LED1 pad 4: unconnected-(LED1-BK-Pad4) -> MCU B
- LED2 pad 1: GND -> VSYS
- LED2 pad 2: MCU R -> LED2
- LED2 pad 3: MCU G -> LED1
- LED2 pad 4: MCU B -> LED0
- MBS0 pad 10: VDD A22 -> VOUT 3.3V
- MBS0 pad 8: VDD A22 -> VOUT 3.3V
- MBS1 pad 4: VDD A22 -> VOUT 3.3V
- MCU1 pad A22: VDD A22 -> 3.3V
- MCU1 pad AD14: VDD A22 -> 3.3V
- MCU1 pad AD23: VDD A22 -> 3.3V
- MCU1 pad B1: VDD A22 -> 3.3V
- MCU1 pad W1: VDD A22 -> 3.3V
- MCU1 pad Y2: VDD A22 -> 3.3V
- R11 pad 1: VBUS -> GND
- R11 pad 2: Net-(LED1-A) -> Net-(ICCPR1-VSET2)
- U1 pad 1: +3V3 -> 3.3V
- U10 pad 1: +3V3 -> 3.3V
- U11 pad 1: +3V3 -> 3.3V
- U12 pad 1: +3V3 -> 3.3V
- U13 pad 1: +3V3 -> 3.3V
- U14 pad 1: +3V3 -> 3.3V
- U15 pad 1: +3V3 -> 3.3V
- U16 pad 1: +3V3 -> 3.3V
- U17 pad 1: +3V3 -> 3.3V
- U18 pad 1: +3V3 -> 3.3V
- U19 pad 1: +3V3 -> 3.3V
- U2 pad 1: +3V3 -> 3.3V
- U20 pad 1: +3V3 -> 3.3V
- U21 pad 1: +3V3 -> 3.3V
- U22 pad 1: +3V3 -> 3.3V
- U23 pad 1: +3V3 -> 3.3V
- U24 pad 1: +3V3 -> 3.3V
- U25 pad 1: +3V3 -> 3.3V
- U26 pad 1: +3V3 -> 3.3V
- U27 pad 1: +3V3 -> 3.3V
- U28 pad 1: +3V3 -> 3.3V
- U29 pad 1: +3V3 -> 3.3V
- U3 pad 1: +3V3 -> 3.3V
- U30 pad 1: +3V3 -> 3.3V
- U31 pad 1: +3V3 -> 3.3V
- U32 pad 1: +3V3 -> 3.3V
- U33 pad 1: +3V3 -> 3.3V
- U34 pad 1: +3V3 -> 3.3V
- U35 pad 1: +3V3 -> 3.3V
- U36 pad 1: +3V3 -> 3.3V
- U37 pad 1: +3V3 -> 3.3V
- U38 pad 1: +3V3 -> 3.3V
- U39 pad 1: +3V3 -> 3.3V
- U4 pad 1: +3V3 -> 3.3V
- U40 pad 1: +3V3 -> 3.3V
- U41 pad 1: +3V3 -> 3.3V
- U42 pad 1: +3V3 -> 3.3V
- U42 pad 2: AM4:10 -> AM4:11
- U43 pad 1: +3V3 -> 3.3V
- U44 pad 1: +3V3 -> 3.3V
- U45 pad 1: +3V3 -> 3.3V
- U46 pad 1: +3V3 -> 3.3V
- U47 pad 1: +3V3 -> 3.3V
- U48 pad 1: +3V3 -> 3.3V
- U49 pad 1: +3V3 -> 3.3V
- U5 pad 1: +3V3 -> 3.3V
- U50 pad 1: +3V3 -> 3.3V
- U51 pad 1: +3V3 -> 3.3V
- U52 pad 1: +3V3 -> 3.3V
- U53 pad 1: +3V3 -> 3.3V
- U54 pad 1: +3V3 -> 3.3V
- U55 pad 1: +3V3 -> 3.3V
- U55 pad 2: AM4:11 -> AM4:12
- U56 pad 1: +3V3 -> 3.3V
- U57 pad 1: +3V3 -> 3.3V
- U58 pad 1: +3V3 -> 3.3V
- U59 pad 1: +3V3 -> 3.3V
- U6 pad 1: +3V3 -> 3.3V
- U60 pad 1: +3V3 -> 3.3V
- U61 pad 1: +3V3 -> 3.3V
- U62 pad 1: +3V3 -> unconnected-(U62-VDD-Pad1)
- U62 pad 3: GND -> unconnected-(U62-GND-Pad3)
- U63 pad 1: +3V3 -> 3.3V
- U64 pad 1: +3V3 -> 3.3V
- U64 pad 2: AM4:12 -> AM4:13
- U65 pad 1: +3V3 -> 3.3V
- U66 pad 1: +3V3 -> 3.3V
- U7 pad 1: +3V3 -> 3.3V
- U8 pad 1: +3V3 -> 3.3V
- U9 pad 1: +3V3 -> 3.3V
Routing:
- net AM4:13: track 0.00 -> 58.9 mm, vias 0 -> 1
- net AM4:11: track 45.7 -> 21.4 mm
- net AM4:10: track 21.7 -> 0.00 mm, vias 1 -> 0
- net VDD A22: track 21.3 -> 0.00 mm, vias 2 -> 0
- net 3.3V: track 4.81 -> 21.3 mm, vias 0 -> 2
- net AM4:12: track 59.7 -> 44.7 mm
- net Net-(PR1-EN): track 8.30 -> 0.00 mm, vias 2 -> 0
- net GND: track 186.8 -> 183.0 mm, vias 49 -> 47
- net Net-(PR1-SW): track 2.82 -> 0.00 mm
Other:
- board size 301.9 x 162.3 mm -> 301.1 x 142.5 mm

Commit message: Third Commit
Kinda add some little changes but still confused on how using the nPM1300
Parts:
- removed LED2: CLV1L-FKB, LED_SMD:LED_Cree-PLCC4_3.2x2.8mm_CCW
- removed R10, R3, R4, R5: 10k, ScottoKeebs_Components:Resistor_0402
- added LED0: LED_SK6812MINI, ScottoKeebs_Components:LED_SK6812MINI, B.Cu at (307.2, 144.2)
- C17: value 4.7µF -> 1µF
- LED1: value CLV1L-FKB -> LED_SK6812MINI; footprint LED_SMD:LED_Cree-PLCC4_3.2x2.8mm_CCW -> ScottoKeebs_Components:LED_SK6812MINI; moved to B.Cu
- R11: value 250k -> 250-500k
- RK1: footprint Rotary_Encoder:RotaryEncoder_Alps_EC11E-Switch_Vertical_H20mm -> HE_Keyswitch:RotaryEncoder_Bourns_Vertical_PEC11J-9220F-S0015
- moved C12 116.3 mm to (285.3, 217.5)
- moved C13 109.6 mm to (280.5, 214.9)
- moved C15 106.6 mm to (288.7, 212.1)
- moved C14 106.6 mm to (283.3, 210.2)
- moved MBS0 106.2 mm to (178.4, 85.7), turned to 90 degrees
- moved C16 96.4 mm to (280.8, 210.2)
- moved C7 89.5 mm to (253.5, 213.8)
- moved C11 85.3 mm to (246.2, 213.6)
- moved C8 71.1 mm to (250.2, 209.7)
- moved C10 71.1 mm to (242.5, 209.7)
- moved C3 68.5 mm to (189.6, 218.3)
- moved C4 68.5 mm to (189.6, 222.3)
- moved CR1 68.5 mm to (189.7, 220.3)
- moved R6 63.5 mm to (250.0, 191.5)
- moved RSW1 63.5 mm to (256.5, 190.1)
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Connections:
- net 2.4GHz MBS renamed 2.4GHz ICCPR
- AM0 pad 10: MCU SELECT0 -> SELECT0
- AM0 pad 11: MCU SELECT1 -> SELECT1
- AM0 pad 13: MCU SELECT3 -> SELECT3
- AM0 pad 14: MCU SELECT2 -> SELECT2
- AM1 pad 10: MCU SELECT0 -> SELECT0
- AM1 pad 11: MCU SELECT1 -> SELECT1
- AM1 pad 13: MCU SELECT3 -> SELECT3
- AM1 pad 14: MCU SELECT2 -> SELECT2
- AM2 pad 10: MCU SELECT0 -> SELECT0
- AM2 pad 11: MCU SELECT1 -> SELECT1
- AM2 pad 13: MCU SELECT3 -> SELECT3
- AM2 pad 14: MCU SELECT2 -> SELECT2
- AM3 pad 10: MCU SELECT0 -> SELECT0
- AM3 pad 11: MCU SELECT1 -> SELECT1
- AM3 pad 13: MCU SELECT3 -> SELECT3
- AM3 pad 14: MCU SELECT2 -> SELECT2
- AM4 pad 10: MCU SELECT0 -> SELECT0
- AM4 pad 11: MCU SELECT1 -> SELECT1
- AM4 pad 13: MCU SELECT3 -> SELECT3
- AM4 pad 14: MCU SELECT2 -> SELECT2
- C17 pad 2: MCU VBUS -> ICCR VBUS
- DBS0 pad 10: USB D- -> USB D+
- DBS0 pad 11: USB CC1 -> USB D-
- DBS0 pad 9: USB D+ -> USB CC1
- DBS1 pad 2: S1 RK -> S2 RK
- DBS1 pad 4: S2 RK -> S1 RK
- F1 pad 1: MCU VBUS -> ICCR VBUS
- ICCPR1 pad 10: unconnected-(ICCPR1-GPIO3-Pad10) -> BT ICCPR
- ICCPR1 pad 2: unconnected-(ICCPR1-PVSS1-Pad2) -> GND
- ICCPR1 pad 21: MCU VBUS -> ICCR VBUS
- ICCPR1 pad 22: MCU VBUS -> unconnected-(ICCPR1-VBUSOUT-Pad22)
- ICCPR1 pad 25: LED0 -> unconnected-(ICCPR1-LED0-Pad25)
- ICCPR1 pad 26: LED1 -> unconnected-(ICCPR1-LED1-Pad26)
- ICCPR1 pad 27: LED2 -> unconnected-(ICCPR1-LED2-Pad27)
- ICCPR1 pad 7: unconnected-(ICCPR1-GPIO0-Pad7) -> Win ICCPR
- ICCPR1 pad 8: BT MBS -> RESET
- LED1 pad 1: GND -> VSYS
- LED1 pad 2: MCU R -> unconnected-(LED1-DOUT-Pad2)
- LED1 pad 3: MCU G -> GND
- LED1 pad 4: MCU B -> Net-(LED0-DOUT)
- MBS0 pad 1: USB CC1 MBS -> USB D- MBS
- MBS0 pad 10: VOUT 3.3V -> 3.3V
- MBS0 pad 2: USB D- MBS -> USB D+ MBS
- MBS0 pad 3: USB D+ MBS -> USB CC1 MBS
- MBS0 pad 5: MCU VBUS -> ICCR VBUS
- MBS0 pad 7: MCU Win -> Win ICCPR
- MBS0 pad 8: VOUT 3.3V -> 3.3V
- MBS0 pad 9: BT MBS -> BT ICCPR
- MBS1 pad 4: VOUT 3.3V -> 3.3V
- MCU1 pad A10: unconnected-(MCU1-P0.29/AIN5-PadA10) -> AM3
- MCU1 pad A12: unconnected-(MCU1-P0.02/AIN0-PadA12) -> AM2
- MCU1 pad A8: unconnected-(MCU1-P0.31/AIN7-PadA8) -> AM4
- MCU1 pad AD10: MCU SELECT0 -> unconnected-(MCU1-P0.15-PadAD10)
- MCU1 pad AD16: MCU SELECT3 -> unconnected-(MCU1-P0.20-PadAD16)
- MCU1 pad AD18: MCU SELECT2 -> SELECT3
- MCU1 pad AD2: MCU VBUS -> unconnected-(MCU1-VBUS-PadAD2)
- MCU1 pad AD20: AM2 -> SELECT2
- MCU1 pad AD8: MCU SELECT1 -> unconnected-(MCU1-P0.13-PadAD8)
- MCU1 pad J1: unconnected-(MCU1-P0.04/AIN2-PadJ1) -> AM0
- MCU1 pad K2: unconnected-(MCU1-P0.05/AIN3-PadK2) -> AM1
- MCU1 pad L1: AM0 -> unconnected-(MCU1-P0.06-PadL1)
- MCU1 pad N1: AM1 -> SELECT1
- MCU1 pad R1: unconnected-(MCU1-P1.09-PadR1) -> SELECT0
- MCU1 pad U24: AM4 -> unconnected-(MCU1-P1.04-PadU24)
- MCU1 pad W24: AM3 -> unconnected-(MCU1-P1.02-PadW24)
- R7 pad 1: MCU Win -> Win ICCPR
- R8 pad 1: BT MBS -> BT ICCPR
Routing:
- net SELECT0: track 0.00 -> 330.0 mm, vias 0 -> 5
- net SELECT1: track 0.00 -> 327.3 mm, vias 0 -> 5
- net MCU SELECT0: track 319.7 -> 0.00 mm, vias 7 -> 0
- net MCU SELECT1: track 315.9 -> 0.00 mm, vias 7 -> 0
- net MCU SELECT2: track 293.0 -> 0.00 mm, vias 5 -> 0
- net SELECT2: track 0.00 -> 292.8 mm, vias 0 -> 5
- net MCU SELECT3: track 287.2 -> 0.00 mm, vias 5 -> 0
- net SELECT3: track 0.00 -> 286.9 mm, vias 0 -> 5
- net GND: track 183.0 -> 156.6 mm, vias 47 -> 27
- net 3.3V: track 21.3 -> 0.00 mm, vias 2 -> 0
- net DEC4: track 15.5 -> 0.00 mm, vias 2 -> 0
- net AM2: track 53.8 -> 69.3 mm
- net AM3: track 114.3 -> 129.6 mm
- net RESET: track 22.2 -> 9.57 mm
- net Net-(LED0-DOUT): track 0.00 -> 11.7 mm
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- added copper zone on F.Cu, net 3.3V
- removed copper zone on F.Cu, net (none)
Other:
- board size 301.1 x 142.5 mm -> 301.1 x 139.3 mm
