File: MB.kicad_sch (KiCad schematic)
At the start: 64 parts

Commit message: Second Commit
new wiring and label
Parts:
- removed C20, C21: 10µF, ScottoKeebs_Components:Capacitor_0402, symbol Device:C_Small
- removed C22: 1µF, ScottoKeebs_Components:Capacitor_0402, symbol Device:C_Small
- removed C23: 100nF, ScottoKeebs_Components:Capacitor_0402, symbol Device:C_Small
- removed ICC1: TP4057, Package_TO_SOT_SMD:SOT-23-6, symbol Battery_Management:TP4057
- removed L1: 1uF, Inductor_SMD:L_0402_1005Metric, symbol Device:L_Small
- removed LED1: CLV1L-FKB, LED_SMD:LED_Cree-PLCC4_3.2x2.8mm_CCW, symbol LED:CLV1L-FKB
- removed PR1: LM3670MF, Package_TO_SOT_SMD:TSOT-23-5, symbol Regulator_Switching:LM3670MF
- removed R12: 1.6k, ScottoKeebs_Components:Resistor_0402, symbol Device:R_Small
- removed SD1: BAT54C, Package_TO_SOT_SMD:SOT-23, symbol Diode:BAT54C
- C1: value 4.7uF -> 1µF
- C2: value 10uF -> 100nF
- R11: value 1k -> 250k
- renumbered LED2 to LED1, LED3 to LED2
Connections:
- net AM4:10 is gone; now on net GND: AM4.21 (I10)
- net VBUS is gone; now on net GND: R11.1
- net 3.3V: now also C12.2, C13.2, C14.2, C15.2, C16.2, DBG3.1, ICCPR1.32 (VOUT2), MCU1.A22 (VDD), MCU1.AD14 (VDD), MCU1.AD23 (VDD), MCU1.B1 (VDD), MCU1.W1 (VDD), MCU1.Y2 (VDDH); no longer C2.2
- net GND: now also ICCPR1.17 (VSET1); no longer AM4.18 (I13), LED2.1 (A)
- net MCU B: no longer LED2.4 (BK)
- net MCU G: no longer LED2.3 (GK)
- net MCU R: no longer LED2.2 (RK)
- net at ESD1.4 (VCC), F1.2: now also C1.2, C2.2
- net at R11.2: now also ICCPR1.16 (VSET2)
- net VSYS: now reaches ICCPR1.20 (VSYS)
- net VSYS: now also LED2.1 (A)
- net LED0: now reaches ICCPR1.25 (LED0)
- net LED0: now also LED2.4 (BK)
- net LED1: now reaches ICCPR1.26 (LED1)
- net LED1: now also LED2.3 (GK)
- net LED2: now reaches ICCPR1.27 (LED2)
- net LED2: now also LED2.2 (RK)
- removed net VDD A22: C12.2, C13.2, C14.2, C15.2, C16.2, DBG3.1, ICCPR1.32 (VOUT2), MBS0.10 (Pin_10), MBS0.8 (Pin_8), MBS1.4 (Pin_4), MCU1.A22 (VDD), MCU1.AD14 (VDD), MCU1.AD23 (VDD), MCU1.B1 (VDD), MCU1.W1 (VDD), MCU1.Y2 (VDDH)
- new net AM4:13: AM4.18 (I13)
- new net VOUT 3.3V: MBS0.10 (Pin_10), MBS0.8 (Pin_8), MBS1.4 (Pin_4)
Other:
- moved on the sheet: LED2

Commit message: Third Commit
Kinda add some little changes but still confused on how using the nPM1300
Parts:
- removed LED1, LED2: CLV1L-FKB, LED_SMD:LED_Cree-PLCC4_3.2x2.8mm_CCW, symbol LED:CLV1L-FKB
- removed R10, R3, R4, R5: 10k, ScottoKeebs_Components:Resistor_0402, symbol Device:R_Small
- added ARF1: Antenna, HE_Keyswitch:2.4GHz-INVERTED-F-ANTENNA, symbol Device:Antenna
- added C20: 1µF, ScottoKeebs_Components:Capacitor_0402, symbol Device:C_Small
- added C21, C22, C23, C24: 10µF, ScottoKeebs_Components:Capacitor_0402, symbol Device:C_Small
- added L1: 2.2µH, symbol Device:L_Small
- added LED0, LED1: LED_SK6812MINI, ScottoKeebs_Components:LED_SK6812MINI, symbol ScottoKeebs:LED_SK6812MINI
- C17: value 4.7µF -> 1µF
- R3: renamed from R11; value 250k -> 250-500k
Connections:
- net MCU Win is gone; now on net Win ICCPR: MBS0.7 (Pin_7), R7.1
- net VOUT 3.3V is gone; now on net 3.3V: MBS0.10 (Pin_10), MBS0.8 (Pin_8), MBS1.4 (Pin_4)
- net 3.3V: no longer ICCPR1.32 (VOUT2)
- net AM0: now also MCU1.J1 (P0.04/AIN2); no longer MCU1.L1 (P0.06)
- net AM1: now also MCU1.K2 (P0.05/AIN3); no longer MCU1.N1 (P0.08)
- net AM2: now also MCU1.A12 (P0.02/AIN0); no longer MCU1.AD20 (P0.24)
- net AM3: now also MCU1.A10 (P0.29/AIN5); no longer MCU1.W24 (P1.02)
- net AM4: now also MCU1.A8 (P0.31/AIN7); no longer MCU1.U24 (P1.04)
- net GND: now also ICCPR1.2 (PVSS1), LED0.3 (VSS), LED1.3 (VSS)
- net RESET: now also ICCPR1.8 (GPIO1)
- net USB CC1 DBS: now also MBP0.9 (Pin_9); no longer MBP0.11 (Pin_11)
- net USB CC1 MBS: now also MBS0.3 (Pin_3); no longer MBS0.1 (Pin_1)
- net USB D+ DBS: now also MBP0.10 (Pin_10); no longer MBP0.9 (Pin_9)
- net USB D+ MBS: now also MBS0.2 (Pin_2); no longer MBS0.3 (Pin_3)
- net USB D- DBS: now also MBP0.11 (Pin_11); no longer MBP0.10 (Pin_10)
- net USB D- MBS: now also MBS0.1 (Pin_1); no longer MBS0.2 (Pin_2)
- net VSYS: now also LED0.1 (VDD), LED1.1 (VDD)
- net SELECT0: now reaches MCU1.R1 (P1.09)
- net SELECT0: now also AM0.10 (S0), AM1.10 (S0), AM2.10 (S0), AM3.10 (S0), AM4.10 (S0)
- net BT ICCPR: now reaches ICCPR1.10 (GPIO3)
- net BT ICCPR: now also MBS0.9 (Pin_9), R8.1
- net PVDD: now reaches ICCPR1.4 (PVDD)
- net SW2: now reaches ICCPR1.5 (SW2)
- net PVSS2: now reaches ICCPR1.6 (PVSS2)
- net Win ICCPR: now reaches ICCPR1.7 (GPIO0)
- net 2.4GHz MBS renamed 2.4GHz ICCPR
- removed net BT MBS: ICCPR1.8 (GPIO1), MBS0.9 (Pin_9), R8.1
- net LED0: no longer names the net of ICCPR1.25 (LED0)
- net LED1: no longer names the net of ICCPR1.26 (LED1)
- net LED2: no longer names the net of ICCPR1.27 (LED2)
- removed net MCU SELECT0: AM0.10 (S0), AM1.10 (S0), AM2.10 (S0), AM3.10 (S0), AM4.10 (S0), MCU1.AD10 (P0.15)
- net MCU SELECT1 renamed SELECT1
- net SELECT1: now also MCU1.N1 (P0.08); no longer MCU1.AD8 (P0.13)
- net MCU SELECT2 renamed SELECT2
- net SELECT2: now also MCU1.AD20 (P0.24); no longer MCU1.AD18 (P0.22)
- net MCU SELECT3 renamed SELECT3
- net SELECT3: now also MCU1.AD18 (P0.22); no longer MCU1.AD16 (P0.20)
- net MCU VBUS renamed ICCR VBUS
- net ICCR VBUS: no longer ICCPR1.22 (VBUSOUT), MCU1.AD2 (VBUS)
- net RF: no longer names the net of C19.2, L2.2
- net RF: now also ARF1.1 (A)
- new net: LED0.2 (DOUT), LED1.4 (DIN)
- new net MCU LED: LED0.4 (DIN)
- new net VOUT2: ICCPR1.32 (VOUT2)
- no-connect marks 0 -> 11
Other:
- moved on the sheet: C18, C19, L2, R3

Commit message: Fourth Commit
changing some name to not get sued :v
Parts:
- removed ARF1: Antenna, HE_Keyswitch:2.4GHz-INVERTED-F-ANTENNA, symbol Device:Antenna
- removed R6: 10k, ScottoKeebs_Components:Resistor_0402, symbol Device:R_Small
- added C25: 2.2µF, ScottoKeebs_Components:Capacitor_0402, symbol Device:C_Small
- added C26: 100nF, ScottoKeebs_Components:Capacitor_0402, symbol Device:C_Small
- added F2: 900mA, ScottoKeebs_Components:Fuse_0603, symbol Device:Polyfuse_Small
- added R4, R5: 10k, ScottoKeebs_Components:Resistor_0402, symbol Device:R_Small
Connections:
- net USB CC1 DBS is gone; now on net Win DBS: MBP0.9 (Pin_9)
- net USB CC2 DBS is gone; now on net COM OS DBS: MBP0.8 (Pin_8)
- net USB D+ MBS is gone; now on net D+ MBS: ESD1.2 (I/O1), MBS0.2 (Pin_2)
- net USB D- MBS is gone; now on net D- MBS: ESD1.3 (I/O2), MBS0.1 (Pin_1)
- net 2.4GHz ICCPR: now also ICCPR1.11 (GPIO4); no longer ICCPR1.9 (GPIO2)
- net 3.3V: now also MBS0.4 (Pin_4); no longer MBS0.8 (Pin_8)
- net COM OS DBS: no longer MBP0.4 (Pin_4)
- net COM RK DBS: now also MBP1.4 (Pin_4); no longer MBP1.3 (Pin_3)
- net GND: now also ICCPR1.1 (VOUT1), ICCPR1.28 (VINLDO1), ICCPR1.29 (VOUTLDO2), ICCPR1.30 (VINLDO2), ICCPR1.31 (VOUTLDO1), MBP0.4 (Pin_4), MBS0.8 (Pin_8); no longer MBP0.6 (Pin_6), MBS0.6 (Pin_6)
- net ICCR VBUS: now also MBS0.7 (Pin_7); no longer ICCPR1.21 (VBUS), MBS0.5 (Pin_5)
- net MCU VOL DOWN: now also MBS1.1 (Pin_1); no longer MBS1.5 (Pin_5)
- net MCU VOL UP: now also MBS1.2 (Pin_2); no longer MBS1.1 (Pin_1)
- net S2 RK DBS: now also MBP1.1 (Pin_1); no longer MBP1.4 (Pin_4)
- net S2 RK MBS: now also MBS1.5 (Pin_5); no longer MBS1.2 (Pin_2)
- net VBUS DBS: now also MBP0.5 (Pin_5); no longer MBP0.7 (Pin_7)
- net VOL DOWN DBS: now also MBP1.5 (Pin_5); no longer MBP1.1 (Pin_1)
- net VOL UP DBS: now also MBP1.3 (Pin_3); no longer MBP1.5 (Pin_5)
- net Win DBS: no longer MBP0.5 (Pin_5)
- net Win ICCPR: now also ICCPR1.9 (GPIO2), MBS0.3 (Pin_3); no longer ICCPR1.7 (GPIO0), MBS0.7 (Pin_7)
- net SCL: now reaches ICCPR1.13 (SDA)
- net SDA: now reaches ICCPR1.14 (SCL)
- net MCU D+ renamed D+ MBS
- net MCU D- renamed D- MBS
- net USB CC1 MBS renamed CC1 MBS
- net CC1 MBS: now also MBS0.5 (Pin_5); no longer MBS0.3 (Pin_3)
- net USB CC2 MBS renamed CC2 MBS
- net CC2 MBS: now also MBS0.6 (Pin_6); no longer MBS0.4 (Pin_4)
- net USB D+ DBS renamed D+ DBS
- net USB D- DBS renamed D- DBS
- new net CC1 DBS: MBP0.7 (Pin_7)
- new net CC2 DBS: MBP0.6 (Pin_6)
- new net ICCPR VBUS: ICCPR1.21 (VBUS)
- no-connect marks 11 -> 6
Other:
- moved on the sheet: C17, RSW1

Commit message: Fifth Commit
updating track width and via's diameter
Parts:
- removed C20: 1µF, ScottoKeebs_Components:Capacitor_0402, symbol Device:C_Small
- removed C25: 2.2µF, ScottoKeebs_Components:Capacitor_0402, symbol Device:C_Small
- removed R13, R14, R7, R8, R9: 10k, ScottoKeebs_Components:Resistor_0402, symbol Device:R_Small
- added ANT1: ~, symbol HE_Keyswitch:MIFA
- added BAT1: Li-poly, symbol Device:Battery_Cell
- added BP1: Conn_01x02_Pin, symbol Connector:Conn_01x02_Pin
- added C15: 4.7µF, ScottoKeebs_Components:Capacitor_0402, symbol Device:C_Small
- added C23: 2.2µF, ScottoKeebs_Components:Capacitor_0402, symbol Device:C_Small
- added R4, R5, R6: 10k, ScottoKeebs_Components:Resistor_0402, symbol Device:R_Small
- BS1: renamed from Battery1; value Conn_01x02_Socket -> Molex PB 2 pin
- C22: renamed from C23; value 10µF -> 1µF
- L2: renamed from L1; footprint (none) -> Inductor_SMD:L_0805_2012Metric
- renumbered C7 to C1, C15 to C10, C3 to C11, C18 to C12, C19 to C13, C4 to C14, C5 to C16, C6 to C17, C1 to C18, C2 to C19, C8 to C2, C21 to C20, C22 to C21, C17 to C25, C9 to C3, C10 to C4, C11 to C5, C12 to C6, C13 to C7, C16 to C8, C14 to C9, DBG3 to DBG2, DBG4 to DBG3, DBG2 to DBG4, L2 to L1, LED0 to LED1, LED1 to LED2, MBP0 to MBP1, MBP1 to MBP2, MBS0 to MBS1, MBS1 to MBS2, R4 to R7, R5 to R8
Connections:
- net PVDD is gone; now on net VSYS: ICCPR1.4 (PVDD)
- net PVSS2 is gone; now on net GND (using via to GND layer): ICCPR1.6 (PVSS2)
- net S2 RK MBS is gone; now on net GND: MBS2.5 (Pin_5)
- net VOUT2 is gone; now on net 3.3V: ICCPR1.32 (VOUT2)
- net 2.4GHz ICCPR: no longer MBS1.11 (Pin_11)
- net 3.3V: now also C24.2, C26.2, ICCPR1.12 (VDDIO), L2.1, MBS1.2 (Pin_2), MBS1.8 (Pin_8), R7.2, R8.2; no longer MBS1.10 (Pin_10), MBS1.4 (Pin_4), MBS2.4 (Pin_4)
- net BAT: now also C23.2
- net BT ICCPR: no longer MBS1.9 (Pin_9)
- net COM RK DBS: now also MBP2.3 (Pin_3); no longer MBP2.4 (Pin_4)
- net D+ MBS: now also MBS1.10 (Pin_10); no longer MBS1.2 (Pin_2)
- net D- MBS: now also MBS1.11 (Pin_11); no longer MBS1.1 (Pin_1)
- net GND: now also C21.1, C22.1, C25.2, C26.1, ICCPR1.33 (AVSS), MBS1.4 (Pin_4), BAT1.2 (-), BP1.2 (Pin_2), C15.2, C23.1, R4.1, R5.1, R6.1; no longer BS1.2 (Pin_2), C25.1, ICCPR1.1 (VOUT1), MBS1.8 (Pin_8)
- net NTC: now also F2.2
- net RESET: now also ICCPR1.7 (GPIO0); no longer ICCPR1.8 (GPIO1)
- net SCL: now also ICCPR1.14 (SCL), R7.1; no longer ICCPR1.13 (SDA)
- net SDA: now also ICCPR1.13 (SDA), R8.1; no longer ICCPR1.14 (SCL)
- net SW2: now also L2.2
- net VOL UP DBS: now also MBP2.4 (Pin_4); no longer MBP2.3 (Pin_3)
- net VSYS: now also C20.2, C21.2, ICCPR1.1 (VOUT1)
- net Win ICCPR: no longer MBS1.3 (Pin_3)
- net VBUS MCU: now reaches C22.2
- net VBUS MCU: now also ICCPR1.22 (VBUSOUT), MCU1.AD2 (VBUS), C15.1
- net VSET2: now reaches ICCPR1.16 (VSET2), R3.2
- net at C13.2, L1.2: now also ANT1.
- net at F2.1: now also BS1.2 (Pin_2)
- net PVSS2 GND: now reaches C20.1
- net GND (using via to GND layer): now reaches C24.1
- net CC1 MBS renamed CC1 ICCPR
- net CC1 ICCPR: now also MBS1.7 (Pin_7); no longer MBS1.5 (Pin_5)
- net CC2 MBS renamed CC2 ICCPR
- net ICCPR VBUS renamed VBUS ICCPR
- net VBUS ICCPR: now also C25.1, F1.1, MBS1.5 (Pin_5)
- removed net ICCR VBUS: C25.2, F1.1, MBS1.7 (Pin_7)
- net S1 RK DBS renamed D RK DBS
- net S2 RK DBS renamed E RK DBS
- new net: BAT1.1 (+), BP1.1 (Pin_1)
- new net 2.4GHz MBS: MBS1.1 (Pin_1), R4.2
- new net BT MBS: MBS1.3 (Pin_3), R5.2
- new net MCU D RK: MBS2.4 (Pin_4)
- new net Win MBS: MBS1.9 (Pin_9), R6.2
- no-connect marks 6 -> 5
Other:
- moved on the sheet: BS1, C1, C10, C11, C12, C13, C14, C16, C17, C18, C19, C2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

Commit message: Sixth Commit
Almost done. Just need to make sure the field zone and each pin is connected properly
Parts:
- removed CR1: 32MHz, Crystal:Crystal_SMD_2016-4Pin_2.0x1.6mm, symbol Device:Crystal
- added C27, C28, C29: N.C., ScottoKeebs_Components:Capacitor_0402, symbol Device:C_Small
- added C30: 1.5pF, ScottoKeebs_Components:Capacitor_0402, symbol Device:C_Small
- added CR1: 32MHz, HE_Keyswitch:Murata_Crystal_SMD_2016-4Pin_2.0x1.6mm, symbol Device:Crystal_GND24
- added R9: 0R, Resistor_SMD:R_0201_0603Metric, symbol Device:R_Small
- C12, C13: NOTES (none) -> 1pF can also be used
- C15, C20, C21, C22, C23, C24, C25, C4, C5, C6, C7: footprint ScottoKeebs_Components:Capacitor_0402 -> ScottoKeebs_Components:Capacitor_0603
- C2: value 100nF -> 100pF
- C26: footprint ScottoKeebs_Components:Capacitor_0402 -> Capacitor_SMD:C_0201_0603Metric
- F1, F2: value 900mA -> 500mA; footprint ScottoKeebs_Components:Fuse_0603 -> Fuse:Fuse_1206_3216Metric
- ICCPR1: value nPM1300-Datasheet Layout -> nPM1300 Datasheet Layout; footprint Package_DFN_QFN:QFN-32-1EP_5x5mm_P0.5mm_EP3.45x3.45mm -> HE_Keyswitch:Nordic_QFN-32-1EP_5x5mm_P0.5mm_EP3.6x3.6mm_ThermalVias
- MCU1: footprint Package_DFN_QFN:Nordic_AQFN-73-1EP_7x7mm_P0.5mm -> HE_Keyswitch:Nordic_AQFN-73-1EP_7x7mm_P0.5mm_Thermal
- R3, R4, R5, R6, R7, R8: footprint ScottoKeebs_Components:Resistor_0402 -> Resistor_SMD:R_0201_0603Metric
Connections:
- net GND (using via to GND layer) is gone; now on net GND: C24.1, ICCPR1.6 (PVSS2)
- net PVSS2 GND is gone; now on net GND: C20.1
- net VBUS DBS is gone; now on net CC2 DBS: MBP1.5 (Pin_5)
- net 2.4GHz ICCPR: now also MBS1.11 (Pin_11), R4.2
- net 3.3V: now also MBS1.10 (Pin_10), MBS1.4 (Pin_4); no longer MBS1.2 (Pin_2), MBS1.8 (Pin_8)
- net BT ICCPR: now also MBS1.9 (Pin_9), R5.2
- net CC1 DBS: now also MBP1.6 (Pin_6); no longer MBP1.7 (Pin_7)
- net CC1 ICCPR: now also MBS1.6 (Pin_6); no longer MBS1.7 (Pin_7)
- net CC2 DBS: no longer MBP1.6 (Pin_6)
- net CC2 ICCPR: now also MBS1.7 (Pin_7); no longer MBS1.6 (Pin_6)
- net DEC4: now also C29.2
- net DEC5: now also MCU1.N24 (DEC5)
- net GND: now also MBS1.8 (Pin_8), MCU1.74 (GND), C27.1, C28.1, C29.1, C30.1, CR1.2, CR1.4; no longer MBS1.4 (Pin_4)
- net MCU D RK: now also MCU1.AD18 (P0.22)
- net MCU LED: now also MCU1.AC19 (P0.23)
- net MCU VOL DOWN: now also MCU1.AD16 (P0.20)
- net MCU VOL UP: now also MCU1.AC17 (P0.21)
- net RESET: now also ICCPR1.15 (SHPHLD); no longer ICCPR1.7 (GPIO0)
- net SCL: now also MCU1.AD8 (P0.13)
- net SDA: now also MCU1.AC9 (P0.14)
- net SELECT2: now also MCU1.AD22 (P1.00); no longer MCU1.AD20 (P0.24)
- net SELECT3: now also MCU1.AC21 (P0.25); no longer MCU1.AD18 (P0.22)
- net Win ICCPR: now also MBS1.3 (Pin_3), R6.2
- net XC1: now also CR1.3
- net XC2: now also CR1.1
- net at C13.2, L1.2: now also C27.2, R9.1; no longer ANT1.
- net DEC2: now reaches MCU1.A18 (DEC2)
- net DEC2: now also C28.2
- net 2.4GHz MBS renamed MBS D-
- net MBS D-: now also ESD1.3 (I/O2), MCU1.AD4 (D-); no longer R4.2
- removed net BT MBS: MBS1.3 (Pin_3), R5.2
- net D+ DBS renamed DBS D+
- net D+ MBS renamed MBS D+
- net MBS D+: now also MBS1.2 (Pin_2); no longer MBS1.10 (Pin_10)
- net D- DBS renamed DBS D-
- removed net D- MBS: ESD1.3 (I/O2), MBS1.11 (Pin_11), MCU1.AD4 (D-)
- net VBUS ICCPR renamed VBUS
- net VBUS: now also MBP1.7 (Pin_7)
- removed net Win MBS: MBS1.9 (Pin_9), R6.2
- new net: ANT1., C30.2, R9.2
- no-connect marks 5 -> 39
Other:
- note added: "MCU"
- note added: "NOTES"
- note added: "PMIC"
- moved on the sheet: AM0, AM1, AM2, AM3, AM4, ANT1, BAT1, BP1, BS1, C1, C10, C11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
