File: MB.kicad_sch (KiCad schematic)
At the start: 66 parts

Commit message: 8th commit
Some minor tweak
Parts:
- removed MBP1: Conn_01x11_Pin, symbol Connector:Conn_01x11_Pin
- removed MBP2: Conn_01x05_Pin, symbol Connector:Conn_01x05_Pin
Connections:
- net VBUS renamed VBUS ICCPR
Other:
- moved on the sheet: C18, C19, C25, ESD1, F1, MBS1, MBS2

Commit message: 9th commit
some minor tweak + adding production files
Parts:
- removed DBG1: RESET, HE_Keyswitch:TestPoint_Pad_D0.5mm, symbol Connector:TestPoint_Alt
- removed DBG2: VDD, HE_Keyswitch:TestPoint_Pad_D0.5mm, symbol Connector:TestPoint_Alt
- removed DBG3: SWDIO, HE_Keyswitch:TestPoint_Pad_D0.5mm, symbol Connector:TestPoint_Alt
- removed DBG4: SWDCLK, HE_Keyswitch:TestPoint_Pad_D0.5mm, symbol Connector:TestPoint_Alt
- removed DBG5: GND, HE_Keyswitch:TestPoint_Pad_D0.5mm, symbol Connector:TestPoint_Alt
- added J3: TC2050-IDC, Connector:Tag-Connect_TC2050-IDC-NL_2x05_P1.27mm_Vertical, symbol Connector_Generic:Conn_02x05_Counter_Clockwise
- AM0, AM1, AM2, AM3, AM4: LCSC Part (none) -> C98457
- BAT1, BP1: now left out of the parts list
- BS1: value Molex PB 2 pin -> HCZZ0001-2; footprint Connector_Molex:Molex_PicoBlade_53261-0271_1x02-1MP_P1.25mm_Horizontal -> HE_Keyswitch:Hong_Cheng_HCZZ0001-2; LCSC Part (none) -> C7433453
- C27, C28, C29: now not fitted
- CR1: LCSC Part (none) -> C914155
- CR2: LCSC Part (none) -> C97605
- ESD1: LCSC Part (none) -> C41409257
- F1, F2: LCSC Part (none) -> C269112
- ICCPR1: LCSC Part (none) -> C7501206
- L1: LCSC Part (none) -> C3249625
- L2: LCSC Part (none) -> C5185544
- LED1, LED2: LCSC Part (none) -> C5149201
- MBS1: value Conn_01x11_Socket -> HCZZ0001-11; footprint Connector_Molex:Molex_PicoBlade_53261-1171_1x11-1MP_P1.25mm_Horizontal -> HE_Keyswitch:Hong_Cheng_HCZZ0001-11; LCSC Part (none) -> C7433462
- MBS2: value Conn_01x05_Socket -> HCZZ0001-5; footprint Connector_Molex:Molex_PicoBlade_53261-0571_1x05-1MP_P1.25mm_Horizontal -> HE_Keyswitch:Hong_Cheng_HCZZ0001-5; LCSC Part (none) -> C7433456
- RSW1: LCSC Part (none) -> C2886897
Connections:
- net 3.3V: now also J3.1 (Pin_1)
- net AM1: now also MCU1.L1 (P0.06)
- net GND: now also J3.3 (Pin_3)
- net MCU D RK: now also MCU1.AD20 (P0.24); no longer MCU1.AD18 (P0.22)
- net MCU LED: now also MCU1.AD22 (P1.00); no longer MCU1.AC19 (P0.23)
- net MCU VOL UP: now also MCU1.AD18 (P0.22); no longer MCU1.AC17 (P0.21)
- net RESET: now also MCU1.AD12 (P0.17)
- net SDA: now also MCU1.AD10 (P0.15); no longer MCU1.AC9 (P0.14)
- net SELECT2: now also MCU1.U24 (P1.04); no longer MCU1.AD22 (P1.00)
- net SELECT3: now also MCU1.W24 (P1.02); no longer MCU1.AC21 (P0.25)
- net SWDCLK: now also J3.4 (Pin_4)
- net SWDIO: now also J3.2 (Pin_2)
- net VBUS ICCPR: now also J3.5 (Pin_5)
- no-connect marks 40 -> 43
Other:
- note added: "Find the 3000mAh one"
- moved on the sheet: AM0, AM1, AM2, AM3, AM4, ANT1, BAT1, BP1, BS1, C1, C10, C11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
