File: HE_Keyboard_Trial.kicad_pcb (KiCad board)
At the start: 2 copper layers, 301.1 x 139.3 mm, 194 parts, among them U1 Hall_Sensor, U10 Hall_Sensor, U11 Hall_Sensor, U12 Hall_Sensor, U13 Hall_Sensor, U14 Hall_Sensor, U15 Hall_Sensor, U16 Hall_Sensor, U17 Hall_Sensor, U18 Hall_Sensor, U19 Hall_Sensor, U2 Hall_Sensor, U20 Hall_Sensor, U21 Hall_Sensor, U22 Hall_Sensor, U23 Hall_Sensor, U24 Hall_Sensor, U25 Hall_Sensor, U26 Hall_Sensor, U27 Hall_Sensor, U28 Hall_Sensor, U29 Hall_Sensor, U3 Hall_Sensor, U30 Hall_Sensor, U31 Hall_Sensor, U32 Hall_Sensor, U33 Hall_Sensor, U34 Hall_Sensor, U35 Hall_Sensor, U36 Hall_Sensor, U37 Hall_Sensor, U38 Hall_Sensor, U39 Hall_Sensor, U4 Hall_Sensor, U40 Hall_Sensor, U41 Hall_Sensor, U42 Hall_Sensor, U43 Hall_Sensor, U44 Hall_Sensor, U45 Hall_Sensor, U46 Hall_Sensor, U47 Hall_Sensor, U48 Hall_Sensor, U49 Hall_Sensor, U5 Hall_Sensor, U50 Hall_Sensor, U51 Hall_Sensor, U52 Hall_Sensor, U53 Hall_Sensor, U54 Hall_Sensor, U55 Hall_Sensor, U56 Hall_Sensor, U57 Hall_Sensor, U58 Hall_Sensor, U59 Hall_Sensor, U6 Hall_Sensor, U60 Hall_Sensor, U61 Hall_Sensor, U62 Hall_Sensor, U63 Hall_Sensor, U64 Hall_Sensor, U65 Hall_Sensor, U66 Hall_Sensor, U7 Hall_Sensor, U8 Hall_Sensor, U9 Hall_Sensor

Commit message: Fourth Commit
changing some name to not get sued :v
Parts:
- removed R11: 250-500k, ScottoKeebs_Components:Resistor_0402
- removed R6: 10k, ScottoKeebs_Components:Resistor_0402
- added C20: 1µF, ScottoKeebs_Components:Capacitor_0402, B.Cu at (272.4, 245.1)
- added C21: 10µF, ScottoKeebs_Components:Capacitor_0402, B.Cu at (272.4, 247.0)
- added C22: 10µF, ScottoKeebs_Components:Capacitor_0402, B.Cu at (272.4, 249.0)
- added C23: 10µF, ScottoKeebs_Components:Capacitor_0402, B.Cu at (272.4, 251.0)
- added C24: 10µF, ScottoKeebs_Components:Capacitor_0402, B.Cu at (272.4, 253.0)
- added C25: 2.2µF, ScottoKeebs_Components:Capacitor_0402, B.Cu at (272.4, 254.9)
- added C26: 100nF, ScottoKeebs_Components:Capacitor_0402, B.Cu at (272.4, 256.9)
- added F2: 900mA, ScottoKeebs_Components:Fuse_0603, B.Cu at (266.0, 245.3)
- added R3: 250-500k, ScottoKeebs_Components:Resistor_0402, B.Cu at (269.5, 245.1)
- added R4: 10k, ScottoKeebs_Components:Resistor_0402, B.Cu at (269.5, 247.1)
- added R5: 10k, ScottoKeebs_Components:Resistor_0402, B.Cu at (269.5, 249.1)
- moved R2 81.8 mm to (70.0, 31.7), turned to 90 degrees
- moved R1 79.0 mm to (68.7, 33.7)
- moved SSW1 78.9 mm to (107.5, 27.3)
- moved SSW2 78.9 mm to (86.4, 27.3)
- moved USB1 78.9 mm to (70.6, 24.5)
- moved DBS0 78.5 mm to (105.6, 33.4)
- moved RK1 52.9 mm to (34.1, 28.2)
- moved DBS1 42.2 mm to (36.3, 33.5), turned to 180 degrees
- moved AM3:2 1.64 mm to (296.0, 112.8)
- moved AM3:9 1.64 mm to (272.2, 93.7)
- moved AM4:13 1.64 mm to (319.8, 150.9)
- moved FID3 1.64 mm to (321.6, 100.8)
- moved H3 1.64 mm to (346.5, 88.6)
- moved U25 1.64 mm to (272.2, 93.7)
- moved U41 1.64 mm to (296.0, 112.8)
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Connections:
- net /Main Board/RF renamed Net-(C19-Pad2)
- DBS0 pad 4: COM OS -> GND
- DBS0 pad 5: Win -> VBUS
- DBS0 pad 6: GND -> USB CC2
- DBS0 pad 7: VBUS -> USB CC1
- DBS0 pad 8: USB CC2 -> COM OS
- DBS0 pad 9: USB CC1 -> Win
- DBS1 pad 1: VOL DOWN -> S2 RK
- DBS1 pad 2: S2 RK -> S1 RK
- DBS1 pad 3: COM RK -> VOL UP
- DBS1 pad 4: S1 RK -> COM RK
- DBS1 pad 5: VOL UP -> VOL DOWN
- ESD1 pad 2: USB D+ MBS -> D+ MBS
- ESD1 pad 3: USB D- MBS -> D- MBS
- ICCPR1 pad 1: unconnected-(ICCPR1-VOUT1-Pad1) -> GND
- ICCPR1 pad 11: unconnected-(ICCPR1-GPIO4-Pad11) -> 2.4GHz ICCPR
- ICCPR1 pad 13: unconnected-(ICCPR1-SDA-Pad13) -> SCL
- ICCPR1 pad 14: unconnected-(ICCPR1-SCL-Pad14) -> SDA
- ICCPR1 pad 21: ICCR VBUS -> ICCPR VBUS
- ICCPR1 pad 23: USB CC1 MBS -> CC1 MBS
- ICCPR1 pad 24: USB CC2 MBS -> CC2 MBS
- ICCPR1 pad 28: unconnected-(ICCPR1-VINLDO1-Pad28) -> GND
- ICCPR1 pad 29: unconnected-(ICCPR1-VOUTLDO2-Pad29) -> GND
- ICCPR1 pad 30: unconnected-(ICCPR1-VINLDO2-Pad30) -> GND
- ICCPR1 pad 31: unconnected-(ICCPR1-VOUTLDO1-Pad31) -> GND
- ICCPR1 pad 32: 3.3V -> VOUT2
- ICCPR1 pad 4: unconnected-(ICCPR1-PVDD-Pad4) -> PVDD
- ICCPR1 pad 5: unconnected-(ICCPR1-SW2-Pad5) -> SW2
- ICCPR1 pad 6: unconnected-(ICCPR1-PVSS2-Pad6) -> PVSS2
- ICCPR1 pad 7: Win ICCPR -> unconnected-(ICCPR1-GPIO0-Pad7)
- ICCPR1 pad 9: 2.4GHz ICCPR -> Win ICCPR
- MBS0 pad 1: USB D- MBS -> D- MBS
- MBS0 pad 2: USB D+ MBS -> D+ MBS
- MBS0 pad 3: USB CC1 MBS -> Win ICCPR
- MBS0 pad 4: USB CC2 MBS -> 3.3V
- MBS0 pad 5: ICCR VBUS -> CC1 MBS
- MBS0 pad 6: GND -> CC2 MBS
- MBS0 pad 7: Win ICCPR -> ICCR VBUS
- MBS0 pad 8: 3.3V -> GND
- MBS1 pad 1: MCU VOL UP -> MCU VOL DOWN
- MBS1 pad 2: S2 RK MBS -> MCU VOL UP
- MBS1 pad 5: MCU VOL DOWN -> S2 RK MBS
- MCU1 pad AD4: MCU D- -> D- MBS
- MCU1 pad AD6: MCU D+ -> D+ MBS
Routing:
- net S2 RK: track 16.9 -> 5.23 mm
- net S1 RK: track 16.9 -> 6.82 mm
- net VOL UP: track 3.42 -> 13.3 mm
- net USB CC2: track 39.7 -> 49.5 mm, vias 0 -> 3
- net GND: track 156.6 -> 164.5 mm, vias 27 -> 29
- net VBUS: track 45.1 -> 51.3 mm, vias 0 -> 2
- net USB D-: track 35.8 -> 41.8 mm
- net COM RK: track 5.50 -> 11.4 mm
- net USB CC1: track 37.7 -> 43.5 mm, vias 0 -> 3
- net COM OS: track 27.6 -> 22.4 mm
- net Win: track 29.1 -> 24.7 mm
- net VOL DOWN: track 3.42 -> 7.17 mm
- net USB D+: track 38.2 -> 41.8 mm
- net COM Mode: track 3.93 -> 2.96 mm
- net 2.4GHz Switch: track 3.82 -> 2.85 mm
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- added copper zone on In1.Cu, net (none)
- added copper zone on In2.Cu, net (none)
- added copper zone on B.Cu, net 3.3V
- added copper zone on In1.Cu, net VBUS
- added copper zone on In2.Cu, net VBUS
- removed copper zone on B.Cu, net VBUS
Other:
- board size 301.1 x 139.3 mm -> 341.5 x 138.1 mm
- copper layers 2 -> 4

Commit message: Fifth Commit
updating track width and via's diameter
Parts:
- removed Battery1: Conn_01x02_Socket, Connector_Molex:Molex_PicoBlade_53261-0271_1x02-1MP_P1.25mm_Horizontal
- removed C3: 12pF, ScottoKeebs_Components:Capacitor_0402
- removed LED0: LED_SK6812MINI, ScottoKeebs_Components:LED_SK6812MINI
- removed MBS0: Conn_01x11_Socket, Connector_Molex:Molex_PicoBlade_53261-1171_1x11-1MP_P1.25mm_Horizontal
- removed R13, R14, R9: 10k, ScottoKeebs_Components:Resistor_0402
- added BS1: Molex PB 2 pin, Connector_Molex:Molex_PicoBlade_53261-0271_1x02-1MP_P1.25mm_Horizontal, F.Cu at (271.1, 200.0)
- added C9: 100nF, ScottoKeebs_Components:Capacitor_0402, F.Cu at (270.2, 206.7)
- added L1: 4.7nH, Inductor_SMD:L_0402_1005Metric, F.Cu at (208.2, 207.1)
- added LED2: LED_SK6812MINI, ScottoKeebs_Components:LED_SK6812MINI, B.Cu at (120.0, 154.8)
- added MBS2: Conn_01x05_Socket, Connector_Molex:Molex_PicoBlade_53261-0571_1x05-1MP_P1.25mm_Horizontal, F.Cu at (278.9, 201.9)
- added R6: 10k, ScottoKeebs_Components:Resistor_0402, F.Cu at (219.6, 237.4)
- AM0, AM1, AM2, AM3, AM4, C2, C21, C24, C26, C8, CR1, CR2, DBG1, DBS0, DBS1, ESD1, F1, F2, ICCPR1, MCU1, R1, R2, R3, R4, R5, R7, R8, RSW1, SSW1, SSW2, USB1: moved to F.Cu
- AM0:0, AM0:1, AM0:10, AM0:11, AM0:12, AM0:13, AM0:14, AM0:15, AM0:2, AM0:3, AM0:4, AM0:5, AM0:6, AM0:7, AM0:8, AM0:9, AM1:0, AM1:1, AM1:10, AM1:11, AM1:12, AM1:14, AM1:15, AM1:2, AM1:3, AM1:5, AM1:6, AM1:7, AM1:8, AM1:9, AM2:0, AM2:1, AM2:13, AM2:14, AM2:15, AM2:2, AM2:4, AM2:5, AM2:6, AM2:7, AM2:8, AM2:9, AM3:0, AM3:1, AM3:12, AM3:13, AM3:14, AM3:15, AM3:2, AM3:4, AM3:5, AM3:6, AM3:7, AM3:8, AM3:9, AM4:0, AM4:1, AM4:11, AM4:12, AM4:13, AM4:14, AM4:15, AM4:2, AM4:7, AM4:8, AM4:9, FID1, FID2, FID3, H1, H2, H3, H4, RK1: moved to B.Cu
- C1, C10: value 1µF -> 100nF; moved to F.Cu
- C11: value 4.7µF -> 12pF; moved to F.Cu
- C12: value 1µF -> 0.8pF; moved to F.Cu
- C13: value 4.7µF -> 0.5pF; moved to F.Cu
- C14, C16: value 100nF -> 12pF; moved to F.Cu
- C15, C7: value 100nF -> 4.7µF; moved to F.Cu
- C17: value 1µF -> 12pF; moved to F.Cu
- C18: value 0.8pF -> 1µF; moved to F.Cu
- C19: value 0.5pF -> 100nF; moved to F.Cu
- C20: value 1µF -> 10µF; moved to F.Cu
- C22: value 10µF -> 1µF; moved to F.Cu
- C23: value 10µF -> 2.2µF; moved to F.Cu
- C25: value 2.2µF -> 1µF; moved to F.Cu
- C4, C6: value 12pF -> 1µF; moved to F.Cu
- C5: value 12pF -> 4.7µF; moved to F.Cu
- DBG2: value SWDCLK -> VDD; moved to F.Cu
- DBG3: value VDD -> SWDIO; moved to F.Cu
- DBG4: value SWDIO -> SWDCLK; moved to F.Cu
- L2: value 4.7nH -> 2.2µH; footprint Inductor_SMD:L_0402_1005Metric -> Inductor_SMD:L_0805_2012Metric; moved to F.Cu
- MBS1: value Conn_01x05_Socket -> Conn_01x11_Socket; footprint Connector_Molex:Molex_PicoBlade_53261-0571_1x05-1MP_P1.25mm_Horizontal -> Connector_Molex:Molex_PicoBlade_53261-1171_1x11-1MP_P1.25mm_Horizontal; moved to F.Cu
- U1, U10, U11, U12, U13, U14, U15, U16, U17, U18, U19, U2, U20, U21, U22, U23, U24, U25, U26, U27, U28, U29, U3, U30, U31, U32, U33, U34, U35, U36, U37, U38, U39, U4, U40, U41, U42, U43, U44, U45, U46, U47, U48, U49, U5, U50, U51, U52, U53, U54, U55, U56, U57, U58, U59, U6, U60, U61, U62, U63, U64, U65, U66, U7, U8, U9: footprint Package_TO_SOT_SMD:SOT-23 -> HE_Keyswitch:GH39FKSW_OH49E-S; moved to B.Cu
- moved RK1 355.5 mm to (389.6, 28.2)
- moved DBS1 351.0 mm to (387.4, 33.5), turned to 0 degrees
- moved FID1 293.8 mm to (359.7, 69.4), turned to 180 degrees
- moved AM4:0 290.3 mm to (67.6, 150.6), turned to 180 degrees
- moved AM4:1 290.3 mm to (67.6, 131.6), turned to 180 degrees
- moved AM4:2 290.3 mm to (67.6, 112.5), turned to 180 degrees
- moved AM4:7 290.3 mm to (67.6, 93.5), turned to 180 degrees
- moved U29 290.3 mm to (67.6, 93.5), turned to 135 degrees
- moved U43 290.3 mm to (67.6, 112.5), turned to 135 degrees
- moved U57 290.3 mm to (67.6, 131.6), turned to 135 degrees
- moved U66 290.3 mm to (67.6, 150.6), turned to 135 degrees
- moved AM0:10 281.2 mm to (353.4, 74.4), turned to 180 degrees
- moved U1 281.2 mm to (353.4, 74.4), turned to 135 degrees
- moved R1 279.2 mm to (347.8, 27.2), turned to 0 degrees
- moved AM0:14 276.4 mm to (351.0, 150.6), turned to 180 degrees
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Connections:
- net Net-(ICCPR1-VSET2) renamed VSET2
- net S1 RK renamed D RK
- net S2 RK renamed E RK
- C1 pad 2: Net-(ESD1-VCC) -> DEC1
- C10 pad 2: DEC4 -> 3.3V
- C11 pad 2: DECUSB -> XC1
- C12 pad 2: 3.3V -> ANT
- C13 pad 2: 3.3V -> Net-(ANT1-Pad)
- C14 pad 2: 3.3V -> XC2
- C15 pad 1: GND -> VBUS MCU
- C15 pad 2: 3.3V -> GND
- C16 pad 2: 3.3V -> XL1
- C17 pad 2: ICCR VBUS -> XL2
- C18 pad 2: ANT -> Net-(ESD1-VCC)
- C19 pad 2: Net-(C19-Pad2) -> Net-(ESD1-VCC)
- C2 pad 2: Net-(ESD1-VCC) -> DEC3
- C20 pad 1: unconnected-(C20-Pad1) -> PVSS2 GND
- C20 pad 2: unconnected-(C20-Pad2) -> VSYS
- C21 pad 1: unconnected-(C21-Pad1) -> GND
- C21 pad 2: unconnected-(C21-Pad2) -> VSYS
- C22 pad 1: unconnected-(C22-Pad1) -> GND
- C22 pad 2: unconnected-(C22-Pad2) -> VBUS MCU
- C23 pad 1: unconnected-(C23-Pad1) -> GND
- C23 pad 2: unconnected-(C23-Pad2) -> BAT
- C24 pad 1: unconnected-(C24-Pad1) -> PVSS2
- C24 pad 2: unconnected-(C24-Pad2) -> 3.3V
- C25 pad 1: unconnected-(C25-Pad1) -> VBUS ICCPR
- C25 pad 2: unconnected-(C25-Pad2) -> GND
- C26 pad 1: unconnected-(C26-Pad1) -> GND
- C26 pad 2: unconnected-(C26-Pad2) -> 3.3V
- C4 pad 2: XC2 -> DEC4
- C5 pad 2: XL1 -> DECUSB
- C6 pad 2: XL2 -> 3.3V
- C7 pad 2: DEC1 -> 3.3V
- C8 pad 2: DEC3 -> 3.3V
- DBG2 pad 1: SWDCLK -> 3.3V
- DBG3 pad 1: 3.3V -> SWDIO
- DBG4 pad 1: SWDIO -> SWDCLK
- F1 pad 1: ICCR VBUS -> VBUS ICCPR
- F2 pad 1: unconnected-(F2-Pad1) -> Net-(BS1-Pin_2)
- F2 pad 2: unconnected-(F2-Pad2) -> NTC
- ICCPR1 pad 1: GND -> VSYS
- ICCPR1 pad 12: unconnected-(ICCPR1-VDDIO-Pad12) -> 3.3V
- ICCPR1 pad 13: SCL -> SDA
- ICCPR1 pad 14: SDA -> SCL
- ICCPR1 pad 21: ICCPR VBUS -> VBUS ICCPR
- ICCPR1 pad 22: unconnected-(ICCPR1-VBUSOUT-Pad22) -> VBUS MCU
- ICCPR1 pad 23: CC1 MBS -> CC1 ICCPR
- ICCPR1 pad 24: CC2 MBS -> CC2 ICCPR
- ICCPR1 pad 32: VOUT2 -> 3.3V
- ICCPR1 pad 33: unconnected-(ICCPR1-AVSS-Pad33) -> GND
- ICCPR1 pad 4: PVDD -> VSYS
- ICCPR1 pad 7: unconnected-(ICCPR1-GPIO0-Pad7) -> RESET
- ICCPR1 pad 8: RESET -> unconnected-(ICCPR1-GPIO1-Pad8)
- L2 pad 1: ANT -> 3.3V
- L2 pad 2: Net-(C19-Pad2) -> SW2
- LED1 pad 2: unconnected-(LED1-DOUT-Pad2) -> Net-(LED1-DOUT)
- LED1 pad 4: Net-(LED0-DOUT) -> MCU LED
- MBS1 pad 1: MCU VOL DOWN -> 2.4GHz MBS
- MBS1 pad 2: MCU VOL UP -> 3.3V
- MBS1 pad 3: GND -> BT MBS
- MBS1 pad 4: 3.3V -> GND
- MBS1 pad 5: S2 RK MBS -> VBUS ICCPR
- MCU1 pad AD2: unconnected-(MCU1-VBUS-PadAD2) -> VBUS MCU
- R4 pad 1: unconnected-(R4-Pad1) -> GND
- R4 pad 2: unconnected-(R4-Pad2) -> 2.4GHz MBS
- R5 pad 1: unconnected-(R5-Pad1) -> GND
- R5 pad 2: unconnected-(R5-Pad2) -> BT MBS
- R7 pad 1: Win ICCPR -> SCL
- R7 pad 2: GND -> 3.3V
- R8 pad 1: BT ICCPR -> SDA
- R8 pad 2: GND -> 3.3V
- U62 pad 1: unconnected-(U62-VDD-Pad1) -> 3.3V
- U62 pad 3: unconnected-(U62-GND-Pad3) -> GND
Routing:
- net AM4: track 187.9 -> 0.00 mm
- net AM0: track 141.4 -> 0.00 mm
- net AM3: track 129.6 -> 0.00 mm
- net GND: track 164.5 -> 54.5 mm, vias 29 -> 18
- net AM1: track 93.0 -> 0.00 mm, vias 2 -> 0
- net SELECT0: track 329.9 -> 248.9 mm
- net SELECT1: track 326.7 -> 245.8 mm
- net AM2: track 69.3 -> 0.00 mm
- net AM4:13: track 58.9 -> 0.00 mm, vias 1 -> 0
- net AM3:1: track 55.3 -> 0.00 mm, vias 1 -> 0
- net AM3:14: track 54.7 -> 0.00 mm, vias 1 -> 0
- net AM4:15: track 53.8 -> 0.00 mm, vias 1 -> 0
- net AM4:0: track 53.2 -> 0.00 mm, vias 1 -> 0
- net SELECT2: track 292.8 -> 247.7 mm
- net AM4:12: track 44.7 -> 0.00 mm, vias 1 -> 0
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- added copper zone on In1.Cu, net GND
- removed copper zone on In1.Cu, net (none)
- removed copper zone on In2.Cu, net (none)
- removed copper zone on B.Cu, net 3.3V
- removed copper zone on F.Cu, net 3.3V
- removed copper zone on B.Cu, net GND
- removed copper zone on In1.Cu, net VBUS
- removed copper zone on In2.Cu, net VBUS
Other:
- board size 341.5 x 138.1 mm -> 339.6 x 166.8 mm

Commit message: Sixth Commit
Almost done. Just need to make sure the field zone and each pin is connected properly
Parts:
- removed R1, R2: 5.1K, ScottoKeebs_Components:Resistor_0402
- removed USB1: USB_C_Receptacle_USB2.0_14P, ScottoKeebs_Components:USB_C_HRO_TYPE-C-31-M-12
- added C27: N.C., ScottoKeebs_Components:Capacitor_0402, F.Cu at (220.7, 153.7)
- added C28: N.C., ScottoKeebs_Components:Capacitor_0402, F.Cu at (229.6, 155.4)
- added C29: N.C., ScottoKeebs_Components:Capacitor_0402, F.Cu at (224.5, 151.9)
- added C3: 820pF, ScottoKeebs_Components:Capacitor_0402, F.Cu at (224.1, 148.3)
- added C30: 1.5pF, ScottoKeebs_Components:Capacitor_0402, F.Cu at (218.2, 153.7)
- added J1: USB_C_Receptacle_USB2.0_14P, ScottoKeebs_Components:USB_C_HRO_TYPE-C-31-M-12, F.Cu at (340.3, 20.5)
- added R9: 0R, Resistor_SMD:R_0201_0603Metric, F.Cu at (219.5, 154.2)
- AM2:8: value 7 & -> U
- AM2:9: value U -> 7 &
- AM3:8: value 0 ) -> P
- AM3:9: value P -> 0 )
- C15, C20, C21, C22, C23, C24, C25, C4, C5, C6, C7: footprint ScottoKeebs_Components:Capacitor_0402 -> ScottoKeebs_Components:Capacitor_0603
- C2: value 100nF -> 100pF
- C26: footprint ScottoKeebs_Components:Capacitor_0402 -> Capacitor_SMD:C_0201_0603Metric
- CR1: footprint Crystal:Crystal_SMD_2016-4Pin_2.0x1.6mm -> HE_Keyswitch:Murata_Crystal_SMD_2016-4Pin_2.0x1.6mm
- F1, F2: value 900mA -> 500mA; footprint ScottoKeebs_Components:Fuse_0603 -> Fuse:Fuse_1206_3216Metric
- ICCPR1: value nPM1300-Datasheet Layout -> nPM1300 Datasheet Layout; footprint Package_DFN_QFN:QFN-32-1EP_5x5mm_P0.5mm_EP3.45x3.45mm -> HE_Keyswitch:Nordic_QFN-32-1EP_5x5mm_P0.5mm_EP3.6x3.6mm_ThermalVias
- LED1, LED2: moved to F.Cu
- MCU1: footprint Package_DFN_QFN:Nordic_AQFN-73-1EP_7x7mm_P0.5mm -> HE_Keyswitch:Nordic_AQFN-73-1EP_7x7mm_P0.5mm_Thermal
- R3, R4, R5, R6, R7, R8: footprint ScottoKeebs_Components:Resistor_0402 -> Resistor_SMD:R_0201_0603Metric
- moved C25 180.7 mm to (227.6, 91.2), turned to 90 degrees
- moved C26 179.1 mm to (232.4, 97.2), turned to 180 degrees
- moved C23 178.4 mm to (230.5, 91.2), turned to -90 degrees
- moved MBS2 178.1 mm to (143.4, 86.3)
- moved C22 174.7 mm to (226.1, 91.2), turned to -90 degrees
- moved C21 174.2 mm to (229.0, 91.2), turned to -90 degrees
- moved C24 169.9 mm to (230.9, 102.8), turned to -90 degrees
- moved F2 167.9 mm to (176.5, 78.5), turned to 90 degrees
- moved ESD1 164.7 mm to (244.3, 77.0), turned to 0 degrees
- moved F1 159.6 mm to (249.2, 74.7), turned to -90 degrees
- moved R6 151.1 mm to (242.4, 88.1), turned to 90 degrees
- moved BS1 150.9 mm to (181.1, 78.9), turned to 90 degrees
- moved R3 148.7 mm to (232.4, 94.7), turned to 180 degrees
- moved R5 148.1 mm to (234.9, 88.1), turned to 90 degrees
- moved R4 146.2 mm to (232.1, 87.8)
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Connections:
- C20 pad 1: PVSS2 GND -> GND
- C24 pad 1: PVSS2 -> GND
- C25 pad 1: VBUS ICCPR -> VBUS
- CR1 pad 2: XC1 -> GND
- CR1 pad 3: (no net) -> XC1
- CR1 pad 4: (no net) -> GND
- DBS0 pad 5: VBUS -> USB CC2
- DBS0 pad 6: USB CC2 -> USB CC1
- DBS0 pad 7: USB CC1 -> VBUS
- DBS1 pad 1: E RK -> GND
- DBS1 pad 4: COM RK -> GND
- ESD1 pad 2: D+ MBS -> MBS D+
- ESD1 pad 3: D- MBS -> MBS D-
- F1 pad 1: VBUS ICCPR -> VBUS
- ICCPR1 pad 15: unconnected-(ICCPR1-SHPHLD-Pad15) -> RESET
- ICCPR1 pad 21: VBUS ICCPR -> VBUS
- ICCPR1 pad 6: PVSS2 -> GND
- ICCPR1 pad 7: RESET -> unconnected-(ICCPR1-GPIO0-Pad7)
- MBS1 pad 1: 2.4GHz MBS -> MBS D-
- MBS1 pad 10: D+ MBS -> 3.3V
- MBS1 pad 11: D- MBS -> 2.4GHz ICCPR
- MBS1 pad 2: 3.3V -> MBS D+
- MBS1 pad 3: BT MBS -> Win ICCPR
- MBS1 pad 4: GND -> 3.3V
- MBS1 pad 5: VBUS ICCPR -> VBUS
- MBS1 pad 6: CC2 ICCPR -> CC1 ICCPR
- MBS1 pad 7: CC1 ICCPR -> CC2 ICCPR
- MBS1 pad 8: 3.3V -> GND
- MBS1 pad 9: Win MBS -> BT ICCPR
- MCU1 pad A18: unconnected-(MCU1-DEC2-PadA18) -> DEC2
- MCU1 pad AC17: unconnected-(MCU1-P0.21-PadAC17) -> MCU VOL UP
- MCU1 pad AC19: unconnected-(MCU1-P0.23-PadAC19) -> MCU LED
- MCU1 pad AC21: unconnected-(MCU1-P0.25-PadAC21) -> SELECT3
- MCU1 pad AC9: unconnected-(MCU1-P0.14-PadAC9) -> SDA
- MCU1 pad AD16: unconnected-(MCU1-P0.20-PadAD16) -> MCU VOL DOWN
- MCU1 pad AD18: SELECT3 -> MCU D RK
- MCU1 pad AD20: SELECT2 -> unconnected-(MCU1-P0.24-PadAD20)
- MCU1 pad AD22: unconnected-(MCU1-P1.00-PadAD22) -> SELECT2
- MCU1 pad AD4: D- MBS -> MBS D-
- MCU1 pad AD6: D+ MBS -> MBS D+
- MCU1 pad AD8: unconnected-(MCU1-P0.13-PadAD8) -> SCL
- MCU1 pad N24: unconnected-(MCU1-DEC5-PadN24) -> DEC5
- R4 pad 2: 2.4GHz MBS -> 2.4GHz ICCPR
- R5 pad 2: BT MBS -> BT ICCPR
- R6 pad 2: Win MBS -> Win ICCPR
- RK1 pad C: COM RK -> GND
- RK1 pad E: E RK -> GND
- RK1 pad MP: unconnected-(RK1-PadMP) -> MP
- U11 pad 2: AM3:8 -> AM3:9
- U22 pad 2: AM2:9 -> AM2:8
- U25 pad 2: AM3:9 -> AM3:8
- U8 pad 2: AM2:8 -> AM2:9
Routing:
- net AM4: track 0.00 -> 194.9 mm
- net VSYS: track 0.00 -> 168.1 mm, vias 0 -> 5
- net AM3: track 0.00 -> 139.1 mm
- net AM0: track 0.00 -> 132.0 mm
- net MCU VOL DOWN: track 0.00 -> 129.7 mm
- net MCU D RK: track 0.00 -> 129.5 mm
- net MCU VOL UP: track 0.00 -> 129.4 mm
- net AM1: track 0.00 -> 84.3 mm
- net AM2: track 0.00 -> 83.9 mm
- net RESET: track 9.57 -> 86.7 mm, vias 3 -> 6
- net SELECT0: track 248.9 -> 319.7 mm
- net SELECT1: track 245.8 -> 316.3 mm
- net VBUS MCU: track 0.00 -> 69.8 mm, vias 0 -> 2
- net 3.3V: track 2.97 -> 71.5 mm, vias 5 -> 10
- net NTC: track 0.00 -> 66.2 mm, vias 0 -> 2
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- removed copper zone on F.Cu, net GND
Other:
- board size 339.6 x 166.8 mm -> 328.6 x 142 mm

Commit message: 7th Commit
Adding the reduced nRF52840 dongle and some minor tweak
Parts:
- removed C15: 4.7µF, ScottoKeebs_Components:Capacitor_0603
- added ANT1: ~, HE_Keyswitch:MIFA, F.Cu at (197.9, 160.5)
- added ANT2: ~, HE_Keyswitch:MIFA, F.Cu at (154.2, 44.9)
- added C31: 12pF, Capacitor_SMD:C_0201_0603Metric, F.Cu at (163.4, 44.0)
- added C32: 12pF, Capacitor_SMD:C_0201_0603Metric, F.Cu at (167.0, 44.0)
- added C33: 100nF, Capacitor_SMD:C_0201_0603Metric, B.Cu at (174.6, 39.1)
- added C34: N.C., Capacitor_SMD:C_0201_0603Metric, B.Cu at (169.1, 43.4)
- added C35: 100pF, Capacitor_SMD:C_0201_0603Metric, B.Cu at (164.9, 41.5)
- added C36: 1µF, ScottoKeebs_Components:Capacitor_0603, B.Cu at (171.9, 44.0)
- added C37: 47nF, Capacitor_SMD:C_0201_0603Metric, B.Cu at (172.2, 42.8)
- added C38: 820pF, Capacitor_SMD:C_0201_0603Metric, B.Cu at (165.2, 38.4)
- added C39: 4.7µF, ScottoKeebs_Components:Capacitor_0603, B.Cu at (175.3, 34.2)
- added C40: N.C., Capacitor_SMD:C_0201_0603Metric, F.Cu at (165.2, 38.0)
- added C41: 12pF, Capacitor_SMD:C_0201_0603Metric, F.Cu at (177.1, 41.5)
- added C42: 12pF, Capacitor_SMD:C_0201_0603Metric, F.Cu at (178.3, 43.8)
- added C43: 1µF, ScottoKeebs_Components:Capacitor_0603, B.Cu at (176.1, 40.2)
- added C44: 0.8pF, Capacitor_SMD:C_0201_0603Metric, F.Cu at (165.1, 40.1)
- added C45: 0.5pF, Capacitor_SMD:C_0201_0603Metric, F.Cu at (162.8, 40.1)
- added C46: N.C., Capacitor_SMD:C_0201_0603Metric, F.Cu at (161.6, 44.6)
- added C47: 1.5pF, Capacitor_SMD:C_0201_0603Metric, F.Cu at (159.3, 44.6)
- added C48: 4.7µF, ScottoKeebs_Components:Capacitor_0603, B.Cu at (174.6, 37.2)
- added C49: 100nF, Capacitor_SMD:C_0201_0603Metric, B.Cu at (167.4, 43.4)
- added C50: 100nF, Capacitor_SMD:C_0201_0603Metric, B.Cu at (169.8, 34.0)
- added C51: 100nF, Capacitor_SMD:C_0201_0603Metric, B.Cu at (167.2, 34.0)
- added C52: 4.7µF, ScottoKeebs_Components:Capacitor_0402, F.Cu at (176.7, 35.7)
- added C53: 100nF, Capacitor_SMD:C_0201_0603Metric, F.Cu at (176.8, 36.6)
- added C54: 4.7µF, ScottoKeebs_Components:Capacitor_0402, B.Cu at (173.3, 34.3)
- added C57: N.C., Capacitor_SMD:C_0201_0603Metric, F.Cu at (164.3, 38.0)
- added C58: 10nF, Capacitor_SMD:C_0201_0603Metric, B.Cu at (179.7, 36.2)
- added C59: 100nF, Capacitor_SMD:C_0201_0603Metric, B.Cu at (179.3, 35.1)
- added CR3: 32MHz, HE_Keyswitch:Murata_Crystal_SMD_2016-4Pin_2.0x1.6mm, F.Cu at (165.2, 44.2)
- added CR4: 32.768kHz, Crystal:Crystal_SMD_2012-2Pin_2.0x1.2mm, F.Cu at (178.3, 42.0)
- added DBG5: GND, HE_Keyswitch:TestPoint_Pad_D0.5mm, F.Cu at (208.9, 149.4)
- added ESD2: PRTR5V0U2X, Package_TO_SOT_SMD:SOT-143, F.Cu at (177.8, 38.6)
- added F3: 500mA, Fuse:Fuse_1206_3216Metric, B.Cu at (177.6, 43.3)
- added FB3: 120R/0.85A, Inductor_SMD:L_0201_0603Metric, B.Cu at (178.9, 36.2)
- added FB4: 120R/0.85A, Inductor_SMD:L_0201_0603Metric, B.Cu at (178.8, 33.7)
- added J1: USB_A, HE_Keyswitch:USB A, B.Cu at (188.9, 38.6)
- added J2: TC2050-IDC, Connector:Tag-Connect_TC2050-IDC-NL_2x05_P1.27mm_Vertical, B.Cu at (162.6, 35.4)
- added L3: 4.7nH, Inductor_SMD:L_0201_0603Metric, F.Cu at (163.9, 39.8)
- added L4: 10µH, Inductor_SMD:L_0603_1608Metric, B.Cu at (176.1, 37.2)
- added L5: 10nH, Inductor_SMD:L_0603_1608Metric, B.Cu at (174.6, 41.4)
- added L6: 15nH, Inductor_SMD:L_0402_1005Metric, B.Cu at (174.4, 43.5)
- added MCU2: nRF52840 Datasheet Layout, HE_Keyswitch:Nordic_AQFN-73-1EP_7x7mm_P0.5mm_Thermal, F.Cu at (170.0, 38.6)
- added R1: 0R, Resistor_SMD:R_0201_0603Metric, F.Cu at (160.4, 44.9)
- added R2: 4R7, Resistor_SMD:R_0201_0603Metric, B.Cu at (174.2, 34.4)
- H1, H2, H3, H4: footprint MountingHole:MountingHole_3.2mm_M3_Pad -> MountingHole:MountingHole_2.2mm_M2
- L2: footprint Inductor_SMD:L_0805_2012Metric -> HE_Keyswitch:Samsung_CIGT201610EH2R2MNE
- MCU1: value nRF52840 Datasheet Layout -> nRF52840 aQFN73 Datasheet Layout
- moved RK1 333.4 mm to (59.0, 79.7)
- moved DBS1 325.8 mm to (63.7, 79.7), turned to 90 degrees
- moved DBS0 43.7 mm to (325.9, 68.0)
- moved SSW1 43.7 mm to (324.0, 61.8)
- moved SSW2 43.7 mm to (345.1, 61.8)
- moved USBC1 43.7 mm to (360.8, 59.0)
- moved C11 18.6 mm to (206.9, 161.9), turned to 90 degrees
- moved CR1 18.4 mm to (208.9, 161.8)
- moved C14 18.2 mm to (210.8, 161.7), turned to -90 degrees
- moved C7 17.0 mm to (220.3, 150.8), turned to 90 degrees
- moved C18 16.8 mm to (232.4, 82.9)
- moved C19 16.8 mm to (231.4, 82.9)
- moved C8 16.5 mm to (212.4, 160.7), turned to 180 degrees
- moved L2 16.4 mm to (214.2, 109.3)
- moved DBG1 16.4 mm to (208.9, 147.9)
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- renumbered J1 to USBC1
Connections:
- C1 pad 1: GND -> DEC1
- C1 pad 2: DEC1 -> GND
- C10 pad 1: GND -> 3.3V
- C10 pad 2: 3.3V -> GND
- C11 pad 1: GND -> XC1
- C11 pad 2: XC1 -> GND
- C12 pad 1: GND -> H23
- C12 pad 2: ANT -> GND
- C13 pad 1: GND -> Net-(C13-Pad1)
- C13 pad 2: Net-(C13-Pad2) -> GND
- C14 pad 1: GND -> XC2
- C14 pad 2: XC2 -> GND
- C16 pad 1: GND -> XL1
- C16 pad 2: XL1 -> GND
- C17 pad 1: GND -> XL2
- C17 pad 2: XL2 -> GND
- C18 pad 1: GND -> Net-(ESD1-VCC)
- C18 pad 2: Net-(ESD1-VCC) -> GND
- C19 pad 1: GND -> Net-(ESD1-VCC)
- C19 pad 2: Net-(ESD1-VCC) -> GND
- C2 pad 1: GND -> DEC3
- C2 pad 2: DEC3 -> GND
- C20 pad 1: GND -> VSYS
- C20 pad 2: VSYS -> GND
- C21 pad 1: GND -> VSYS
- C21 pad 2: VSYS -> GND
- C22 pad 1: GND -> VBUSOUT
- C22 pad 2: VBUS MCU -> GND
- C23 pad 1: GND -> BAT
- C23 pad 2: BAT -> GND
- C24 pad 1: GND -> 3.3V
- C24 pad 2: 3.3V -> GND
- C26 pad 1: GND -> 3.3V
- C26 pad 2: 3.3V -> GND
- C27 pad 1: GND -> Net-(C13-Pad1)
- C27 pad 2: Net-(C13-Pad2) -> GND
- C28 pad 1: GND -> DEC2
- C28 pad 2: DEC2 -> GND
- C29 pad 1: GND -> DEC4
- C29 pad 2: DEC4 -> GND
- C3 pad 1: GND -> DEC5
- C3 pad 2: DEC5 -> GND
- C30 pad 1: GND -> Net-(ANT1-Pad1)
- C30 pad 2: Net-(ANT1-Pad) -> GND
- C4 pad 1: GND -> DEC4
- C4 pad 2: DEC4 -> GND
- C5 pad 1: GND -> DECUSB
- C5 pad 2: DECUSB -> GND
- C6 pad 1: GND -> 3.3V
- C6 pad 2: 3.3V -> GND
- C7 pad 1: GND -> 3.3V
- C7 pad 2: 3.3V -> GND
- C8 pad 1: GND -> 3.3V
- C8 pad 2: 3.3V -> GND
- C9 pad 1: GND -> 3.3V
- C9 pad 2: 3.3V -> GND
- DBS1 pad 1: GND -> VOL DOWN
- DBS1 pad 2: D RK -> GND
- DBS1 pad 3: VOL UP -> D RK
- DBS1 pad 5: VOL DOWN -> VOL UP
- ICCPR1 pad 22: VBUS MCU -> VBUSOUT
- L1 pad 1: ANT -> H23
- L1 pad 2: Net-(C13-Pad2) -> Net-(C13-Pad1)
- MCU1 pad AD2: VBUS MCU -> unconnected-(MCU1-VBUS-PadAD2)
- MCU1 pad H23: ANT -> H23
- R3 pad 1: GND -> VSET2
- R3 pad 2: VSET2 -> GND
- R4 pad 1: GND -> 2.4GHz ICCPR
- R4 pad 2: 2.4GHz ICCPR -> GND
- R5 pad 1: GND -> BT ICCPR
- R5 pad 2: BT ICCPR -> GND
- R6 pad 1: GND -> Win ICCPR
- R6 pad 2: Win ICCPR -> GND
- R9 pad 1: Net-(C13-Pad2) -> Net-(C13-Pad1)
- R9 pad 2: Net-(ANT1-Pad) -> Net-(ANT1-Pad1)
Routing:
- net GND: track 106.4 -> 254.9 mm, vias 44 -> 218
- net MCU LED: track 0.00 -> 115.4 mm, vias 0 -> 2
- net VBUS MCU: track 69.8 -> 0.00 mm, vias 2 -> 0
- net VBUS ESD: track 0.00 -> 55.9 mm, vias 0 -> 2
- net Net-(ANT1-Pad1): track 0.00 -> 32.1 mm
- net Net-(ANT2-Pad1): track 0.00 -> 32.0 mm
- net Net-(ANT1-Pad): track 31.1 -> 0.00 mm
- net Dongle D-: track 0.00 -> 24.5 mm, vias 0 -> 1
- net Dongle D+: track 0.00 -> 23.4 mm, vias 0 -> 1
- net VSYS: track 168.1 -> 181.5 mm, vias 5 -> 7
- net Dongle DEC4: track 0.00 -> 12.6 mm, vias 0 -> 2
- net Net-(ESD2-VCC): track 0.00 -> 11.9 mm, vias 0 -> 1
- net Dongle XL2: track 0.00 -> 10.5 mm
- net VOL UP: track 13.6 -> 5.05 mm
- net MBS D+: track 65.1 -> 72.9 mm
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- added copper zone on B.Cu, net 3.3V
- added copper zone on F.Cu, net 3.3V
- added copper zone on B.Cu, net GND
- added copper zone on F.Cu, net GND
- removed copper zone on In1.Cu, net GND
Other:
- board size 328.6 x 142 mm -> 319.9 x 132.1 mm
- copper layers 4 -> 2
