File: HE_Keyboard_Trial.kicad_pcb (KiCad board)
At the start: 2 copper layers, 319.9 x 132.1 mm, 250 parts, among them J1 USB_A, J2 TC2050-IDC, U1 Hall_Sensor, U10 Hall_Sensor, U11 Hall_Sensor, U12 Hall_Sensor, U13 Hall_Sensor, U14 Hall_Sensor, U15 Hall_Sensor, U16 Hall_Sensor, U17 Hall_Sensor, U18 Hall_Sensor, U19 Hall_Sensor, U2 Hall_Sensor, U20 Hall_Sensor, U21 Hall_Sensor, U22 Hall_Sensor, U23 Hall_Sensor, U24 Hall_Sensor, U25 Hall_Sensor, U26 Hall_Sensor, U27 Hall_Sensor, U28 Hall_Sensor, U29 Hall_Sensor, U3 Hall_Sensor, U30 Hall_Sensor, U31 Hall_Sensor, U32 Hall_Sensor, U33 Hall_Sensor, U34 Hall_Sensor, U35 Hall_Sensor, U36 Hall_Sensor, U37 Hall_Sensor, U38 Hall_Sensor, U39 Hall_Sensor, U4 Hall_Sensor, U40 Hall_Sensor, U41 Hall_Sensor, U42 Hall_Sensor, U43 Hall_Sensor, U44 Hall_Sensor, U45 Hall_Sensor, U46 Hall_Sensor, U47 Hall_Sensor, U48 Hall_Sensor, U49 Hall_Sensor, U5 Hall_Sensor, U50 Hall_Sensor, U51 Hall_Sensor, U52 Hall_Sensor, U53 Hall_Sensor, U54 Hall_Sensor, U55 Hall_Sensor, U56 Hall_Sensor, U57 Hall_Sensor, U58 Hall_Sensor, U59 Hall_Sensor, U6 Hall_Sensor, U60 Hall_Sensor, U61 Hall_Sensor, U62 Hall_Sensor, U63 Hall_Sensor, U64 Hall_Sensor, U65 Hall_Sensor, U66 Hall_Sensor, U7 Hall_Sensor, U8 Hall_Sensor, U9 Hall_Sensor

Commit message: 8th commit
Some minor tweak
Parts:
- ANT2, C31, C32, C40, C41, C42, C44, C45, C46, C47, C52, C53, C57, CR3, CR4, ESD2, L3, MCU2, R1: moved to B.Cu
- C33, C34, C35, C36, C37, C38, C39, C43, C48, C49, C50, C51, C54, C58, C59, F3, FB3, FB4, J1, J2, L4, L5, L6, R2: moved to F.Cu
- moved SSW2 164.9 mm to (185.4, 103.0)
- moved SSW1 164.9 mm to (164.3, 103.0)
- moved USBC1 164.9 mm to (201.1, 100.2)
- moved DBS0 164.9 mm to (166.2, 109.2)
- moved J1 111.9 mm to (98.6, 104.7)
- moved C58 97.6 mm to (107.9, 102.3)
- moved C59 97.0 mm to (108.3, 101.1), turned to 0 degrees
- moved FB3 96.5 mm to (108.6, 102.3)
- moved FB4 96.3 mm to (108.7, 99.8), turned to 0 degrees
- moved C42 95.6 mm to (109.2, 109.8), turned to 0 degrees
- moved CR4 95.6 mm to (109.2, 108.1)
- moved ESD2 94.9 mm to (109.7, 104.7)
- moved F3 94.5 mm to (110.0, 109.4), turned to 0 degrees
- moved C41 93.8 mm to (110.5, 107.6)
- moved C53 93.4 mm to (110.7, 102.7), turned to 180 degrees
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Connections:
- net VBUS renamed VBUS ICCPR
- MCU2 pad AC13: RST -> unconnected-(MCU2-P0.18/RESET-PadAC13)
- MCU2 pad AC15: RST -> unconnected-(MCU2-P0.19-PadAC15)
- MCU2 pad AC17: RST -> unconnected-(MCU2-P0.21-PadAC17)
- MCU2 pad AC19: RST -> unconnected-(MCU2-P0.23-PadAC19)
- MCU2 pad AC21: RST -> unconnected-(MCU2-P0.25-PadAC21)
- MCU2 pad R24: Dongle P1.06 -> unconnected-(MCU2-P1.06-PadR24)
Routing:
- net GND: track 254.9 -> 275.7 mm, vias 218 -> 232
- net Dongle AD23: track 3.80 -> 6.87 mm
- net VBUS ESD: track 55.9 -> 58.9 mm
- net 3.3V: track 77.4 -> 80.2 mm, vias 67 -> 69
- net Dongle SWDIO: track 3.22 -> 5.30 mm
- net Dongle SWDCLK: track 4.76 -> 6.14 mm
- net Dongle NFC1: track 1.89 -> 2.82 mm
Other:
- board size 319.9 x 132.1 mm -> 301.1 x 109.5 mm
