File: HE_Keyboard_Trial.kicad_pcb (KiCad board)
At the start: 2 copper layers, 301.1 x 109.5 mm, 250 parts, among them J1 USB_A, J2 TC2050-IDC, U1 Hall_Sensor, U10 Hall_Sensor, U11 Hall_Sensor, U12 Hall_Sensor, U13 Hall_Sensor, U14 Hall_Sensor, U15 Hall_Sensor, U16 Hall_Sensor, U17 Hall_Sensor, U18 Hall_Sensor, U19 Hall_Sensor, U2 Hall_Sensor, U20 Hall_Sensor, U21 Hall_Sensor, U22 Hall_Sensor, U23 Hall_Sensor, U24 Hall_Sensor, U25 Hall_Sensor, U26 Hall_Sensor, U27 Hall_Sensor, U28 Hall_Sensor, U29 Hall_Sensor, U3 Hall_Sensor, U30 Hall_Sensor, U31 Hall_Sensor, U32 Hall_Sensor, U33 Hall_Sensor, U34 Hall_Sensor, U35 Hall_Sensor, U36 Hall_Sensor, U37 Hall_Sensor, U38 Hall_Sensor, U39 Hall_Sensor, U4 Hall_Sensor, U40 Hall_Sensor, U41 Hall_Sensor, U42 Hall_Sensor, U43 Hall_Sensor, U44 Hall_Sensor, U45 Hall_Sensor, U46 Hall_Sensor, U47 Hall_Sensor, U48 Hall_Sensor, U49 Hall_Sensor, U5 Hall_Sensor, U50 Hall_Sensor, U51 Hall_Sensor, U52 Hall_Sensor, U53 Hall_Sensor, U54 Hall_Sensor, U55 Hall_Sensor, U56 Hall_Sensor, U57 Hall_Sensor, U58 Hall_Sensor, U59 Hall_Sensor, U6 Hall_Sensor, U60 Hall_Sensor, U61 Hall_Sensor, U62 Hall_Sensor, U63 Hall_Sensor, U64 Hall_Sensor, U65 Hall_Sensor, U66 Hall_Sensor, U7 Hall_Sensor, U8 Hall_Sensor, U9 Hall_Sensor

Commit message: 9th commit
some minor tweak + adding production files
Parts:
- removed DBG1: RESET, HE_Keyswitch:TestPoint_Pad_D0.5mm
- removed DBG2: VDD, HE_Keyswitch:TestPoint_Pad_D0.5mm
- removed DBG3: SWDIO, HE_Keyswitch:TestPoint_Pad_D0.5mm
- removed DBG4: SWDCLK, HE_Keyswitch:TestPoint_Pad_D0.5mm
- removed DBG5: GND, HE_Keyswitch:TestPoint_Pad_D0.5mm
- added J3: TC2050-IDC, Connector:Tag-Connect_TC2050-IDC-NL_2x05_P1.27mm_Vertical, F.Cu at (189.7, 193.7)
- ANT2, C31, C32, C41, C42, C44, C45, C46, C47, C52, C53, CR3, CR4, ESD2, L3, R1: moved to F.Cu
- BS1: value Molex PB 2 pin -> HCZZ0001-2; footprint Connector_Molex:Molex_PicoBlade_53261-0271_1x02-1MP_P1.25mm_Horizontal -> HE_Keyswitch:Hong_Cheng_HCZZ0001-2
- C33, C34, C35, C36, C37, C38, C39, C43, C48, C49, C50, C51, C54, C58, C59, FB3, FB4, J1, J2, L4, L6, R2: moved to B.Cu
- DBS0, MBS1: value Conn_01x11_Socket -> HCZZ0001-11; footprint Connector_Molex:Molex_PicoBlade_53261-1171_1x11-1MP_P1.25mm_Horizontal -> HE_Keyswitch:Hong_Cheng_HCZZ0001-11
- DBS1, MBS2: value Conn_01x05_Socket -> HCZZ0001-5; footprint Connector_Molex:Molex_PicoBlade_53261-0571_1x05-1MP_P1.25mm_Horizontal -> HE_Keyswitch:Hong_Cheng_HCZZ0001-5
- L5: value 10nH -> 10µH; moved to B.Cu
- MCU2: value nRF52840 Datasheet Layout -> nRF52840 aQFN73 Datasheet Layout; moved to F.Cu
- RK1: footprint HE_Keyswitch:RotaryEncoder_Bourns_Vertical_PEC11J-9220F-S0015 -> HE_Keyswitch:RotaryEncoder_CTR_ED11601M-FB15A7.0-C15-202
- SSW1: value MSK13C01 -> K3-1346S-K1; footprint Button_Switch_SMD:SW_SP3T_PCM13 -> HE_Keyswitch:SW_SP3T_Korean_Hroparts_Elec_K3-1346S-K1
- SSW2: value MSK12C01 -> K3-1280S-K1; footprint Button_Switch_SMD:SW_SPDT_PCM12 -> HE_Keyswitch:SW_SPDT_Korean_Hroparts_Elec_K3-1280S-K1
- moved C42 195.0 mm to (303.8, 97.0), turned to -90 degrees
- moved C43 193.2 mm to (304.5, 96.5), turned to 0 degrees
- moved CR4 193.2 mm to (302.1, 96.9), turned to 180 degrees
- moved L6 193.0 mm to (305.9, 100.5), turned to -90 degrees
- moved L5 191.9 mm to (304.7, 99.3)
- moved C41 191.3 mm to (301.6, 98.2), turned to 0 degrees
- moved C33 189.8 mm to (302.6, 96.9), turned to 90 degrees
- moved C36 189.2 mm to (304.7, 102.2), turned to -90 degrees
- moved L4 187.9 mm to (299.3, 96.4), turned to 0 degrees
- moved C58 187.1 mm to (294.9, 96.4), turned to 90 degrees
- moved FB3 187.1 mm to (295.6, 96.4), turned to -90 degrees
- moved C59 187.0 mm to (295.3, 97.6)
- moved C37 186.5 mm to (301.9, 106.4)
- moved C48 186.4 mm to (299.3, 97.9), turned to 0 degrees
- moved C34 186.2 mm to (304.7, 104.2), turned to 0 degrees
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Connections:
- net VSYS renamed /Main Board/VSYS
- DBS0 pad 2: COM Mode -> 3.3V
- DBS0 pad 8: COM OS -> 3.3V
- MCU1 pad AC17: MCU VOL UP -> unconnected-(MCU1-P0.21-PadAC17)
- MCU1 pad AC19: MCU LED -> unconnected-(MCU1-P0.23-PadAC19)
- MCU1 pad AC21: SELECT3 -> unconnected-(MCU1-P0.25-PadAC21)
- MCU1 pad AC9: SDA -> unconnected-(MCU1-P0.14-PadAC9)
- MCU1 pad AD10: unconnected-(MCU1-P0.15-PadAD10) -> SDA
- MCU1 pad AD12: unconnected-(MCU1-P0.17-PadAD12) -> RESET
- MCU1 pad AD18: MCU D RK -> MCU VOL UP
- MCU1 pad AD20: unconnected-(MCU1-P0.24-PadAD20) -> MCU D RK
- MCU1 pad AD22: SELECT2 -> MCU LED
- MCU1 pad L1: unconnected-(MCU1-P0.06-PadL1) -> AM1
- MCU1 pad U24: unconnected-(MCU1-P1.04-PadU24) -> SELECT2
- MCU1 pad W24: unconnected-(MCU1-P1.02-PadW24) -> SELECT3
- MCU2 pad L1: LED 4 -> unconnected-(MCU2-P0.06-PadL1)
- MCU2 pad N1: LED R -> unconnected-(MCU2-P0.08-PadN1)
- MCU2 pad R1: LED G -> unconnected-(MCU2-P1.09-PadR1)
- MCU2 pad U1: LED B -> unconnected-(MCU2-P0.12-PadU1)
- SSW1 pad 3: COM Mode -> 3.3V
- SSW2 pad 2: COM OS -> 3.3V
Routing:
- net VBUS ICCPR: track 86.1 -> 161.7 mm, vias 3 -> 9
- net SWDCLK: track 3.38 -> 29.0 mm, vias 0 -> 2
- net SWDIO: track 3.79 -> 28.2 mm, vias 0 -> 2
- net COM OS: track 22.0 -> 0.00 mm
- net AM4: track 194.9 -> 216.6 mm
- net GND: track 275.7 -> 254.7 mm, vias 232 -> 227
- net RESET: track 85.8 -> 65.0 mm, vias 5 -> 4
- net AM2: track 84.3 -> 101.9 mm
- net VBUS ESD: track 58.9 -> 43.6 mm
- net Net-(C45-Pad1): track 7.85 -> 17.1 mm
- net AM0: track 132.0 -> 141.3 mm
- net Net-(ESD2-VCC): track 11.9 -> 3.92 mm, vias 1 -> 0
- net Net-(J1-GND): track 5.34 -> 11.6 mm
- net MBS D+: track 72.9 -> 67.0 mm
- net MBS D-: track 72.9 -> 67.0 mm
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- added copper zone on F.Cu, net BAT
Other:
- board size 301.1 x 109.5 mm -> 318.7 x 106.4 mm
