File: Dongle.kicad_sch (KiCad schematic)
At the start: 43 parts, among them J1 USB_A, J2 TC2050-IDC

Commit message: 8th commit
Some minor tweak
Connections:
- net Dongle P1.06: no longer names the net of MCU2.R24 (P1.06)
- removed net RST: MCU2.AC13 (P0.18/RESET), MCU2.AC15 (P0.19), MCU2.AC17 (P0.21), MCU2.AC19 (P0.23), MCU2.AC21 (P0.25)
- no-connect marks 38 -> 44
Other:
- moved on the sheet: C52, C53, C58, C59, ESD2, F3, FB3, FB4, J1, J2, MCU2

Commit message: 9th commit
some minor tweak + adding production files
Parts:
- removed MCU2: nRF52840 Datasheet Layout, HE_Keyswitch:Nordic_AQFN-73-1EP_7x7mm_P0.5mm_Thermal, symbol HE_Keyswitch:nRF52840 Datasheet Layout
- added MCU2: nRF52840 aQFN73 Datasheet Layout, HE_Keyswitch:Nordic_AQFN-73-1EP_7x7mm_P0.5mm_Thermal, symbol HE_Keyswitch:nRF52840 aQFN73 Datasheet Layout
- C34, C40, C46, C57: now not fitted
- C35: LCSC Part (none) -> C710791
- C45: LCSC Part (none) -> C2981049
- CR3: LCSC Part (none) -> C914155
- CR4: LCSC Part (none) -> C97603
- ESD2: LCSC Part (none) -> C41409257
- F3: LCSC Part (none) -> C269112
- FB3, FB4: LCSC Part (none) -> C2661865
- L3: LCSC Part (none) -> C86126
- L4: LCSC Part (none) -> C87216
- L5: value 10nH -> 10µH; LCSC Part (none) -> C87216
- L6: LCSC Part (none) -> C87189
Connections:
- net Dongle A22: now also MCU2.A22 (VDD)
- net Dongle AD14: now also MCU2.AD14 (VDD)
- net Dongle AD23: now also MCU2.AD23 (VDD)
- net Dongle B1: now also MCU2.B1 (VDD)
- net Dongle D+: now also MCU2.AD6 (D+)
- net Dongle D-: now also MCU2.AD4 (D-)
- net Dongle DCC: now also MCU2.B3 (DCC)
- net Dongle DCCH: now also MCU2.AB2 (DCCH)
- net Dongle DEC1: now also MCU2.C1 (DEC1)
- net Dongle DEC2: now also MCU2.A18 (DEC2)
- net Dongle DEC3: now also MCU2.D23 (DEC3)
- net Dongle DEC4: now also MCU2.B5 (DEC4), MCU2.E24 (DEC6)
- net Dongle DEC5: now also MCU2.N24 (DEC5)
- net Dongle DECUSB: now also MCU2.AC5 (DECUSB)
- net Dongle H23: now also MCU2.H23 (ANT)
- net Dongle NFC1: now also MCU2.L24 (P0.09/NFC1)
- net Dongle NFC2: now also MCU2.J24 (P0.10/NFC2)
- net Dongle SWDCLK: now also MCU2.AA24 (SWDCLK)
- net Dongle SWDIO: now also MCU2.AC24 (SWDIO)
- net Dongle VDDH: now also MCU2.AD2 (VBUS), MCU2.Y2 (VDDH)
- net Dongle W1: now also MCU2.W1 (VDD)
- net Dongle XC1: now also MCU2.B24 (XC1)
- net Dongle XC2: now also MCU2.A23 (XC2)
- net Dongle XL1: now also MCU2.D2 (P0.00/XL1)
- net Dongle XL2: now also MCU2.F2 (P0.01/XL2)
- net GND: now also MCU2.74 (GND), MCU2.B15 (P1.14), MCU2.B7 (VSS), MCU2.F23 (VSS_PA)
- no-connect marks 44 -> 48
